File: hardware/controlador-flechas-36v/kicad/ControladorFlechas.kicad_pcb (KiCad board)
At the start: 2 copper layers, 105 x 80 mm, 71 parts, among them J1 36V ENTRADA, J2 INTERRUPTOR, J3 FLECHAS, J4 CENTROS, J5 FLORES, J6 BAÑOS, Q1 2N7000, Q2 2N7000, Q3 2N7000, Q4 2N7000, SW2 REINICIO, U1 NE555P, U2 CD4017BE, U3 LM317T, U4 LM317LZ, U5 LM317LZ, U6 LM317LZ

Commit message: PCB: clemas con entrada hacia el borde, serigrafia, un solo puente; ERC/DRC sin errores
Co-Authored-By: Claude Opus 5.5 <noreply@anthropic.com>
Claude-Session: https://claude.ai/code/session_01WVk3oGwfQfGTmAT2PMp8oW
Parts:
- W1: footprint ControladorFlechas:Puente_Alambre_P15.24mm -> ControladorFlechas:Puente_Alambre_P7.62mm
- moved J3 15.2 mm to (56.4, 62.7), turned to -90 degrees
- moved W1 6.73 mm to (143.3, 82.7), turned to 90 degrees
- moved C3 6.48 mm to (132.6, 74.8)
- moved J1 5.08 mm to (149.1, 80.5), turned to 90 degrees
- moved J2 5.08 mm to (149.1, 67.8), turned to 90 degrees
- moved J5 5.08 mm to (64.0, 123.7), turned to 0 degrees
- moved J6 5.08 mm to (76.7, 123.7), turned to 0 degrees
- moved J4 5.08 mm to (136.4, 123.7), turned to 0 degrees
- moved LED6 3.81 mm to (140.5, 79.5)
- moved JP3 3.18 mm to (65.2, 112.9)
- moved R8 2.01 mm to (133.2, 82.7)
- moved C5 0.64 mm to (141.8, 114.8)
- moved F1 0.63 mm to (141.4, 62.7)
Connections:
- J1 pad 1: /VIN -> GND
- J1 pad 2: GND -> /VIN
- J2 pad 1: /VSW -> /VIN
- J2 pad 2: /VIN -> /VSW
- J3 pad 1: /F3N -> +36V
- J3 pad 2: /F2N -> /F1N
- J3 pad 3: /F1N -> /F2N
- J3 pad 4: +36V -> /F3N
- J4 pad 1: /CENT_D -> GND
- J4 pad 2: GND -> /CENT_D
- J5 pad 1: GND -> /V_FLOR
- J5 pad 2: /V_FLOR -> GND
- J6 pad 1: GND -> /V_BANO
- J6 pad 2: /V_BANO -> GND
Routing:
- net GND: track 428.7 -> 437.6 mm
- net +12V: track 95.4 -> 88.3 mm
- net /LED6A: track 4.65 -> 8.99 mm
- net +36V: track 178.7 -> 175.5 mm
- net /V_BANO: track 9.20 -> 12.4 mm
- net /+12V_W1: track 11.0 -> 14.1 mm
- net /TIM: track 39.4 -> 41.4 mm
- net /VSW: track 6.99 -> 7.62 mm
- net /VF: track 8.25 -> 7.62 mm
Other:
- board text added: "+ BAÑOS -"
- board text added: "+ FLORES -"
- board text added: "+36V"
- board text added: "36V+"
- board text added: "CONTROLADOR FLECHAS 36V v1.0"
- board text added: "F1-"
- board text added: "F2-"
- board text added: "F3-"
- board text added: "FLECHAS"
- board text added: "FLECHAS 36V v1.0"
- board text added: "G CENTROS -"
- board text added: "GND"
- board text added: "INTERRUPTOR"
- board text added: "JP2/JP3: NO MONTAR"
- board text added: "LOGICA 12 V"
- board text added: "REINICIO"
- board text added: "SW"
- board text added: "VELOCIDAD"
- board text added: "ZONA 36 V (POTENCIA)"
