File: hardware/controlador-flechas-36v/kicad/ControladorFlechas.kicad_sch (KiCad schematic)
At the start: 71 parts, among them J1 36V ENTRADA, J2 INTERRUPTOR, J3 FLECHAS, J4 CENTROS, J5 FLORES, J6 BAÑOS, Q1 2N7000, Q2 2N7000, Q3 2N7000, Q4 2N7000, SW2 REINICIO, U1 NE555P, U2 CD4017BE, U3 LM317T, U4 LM317LZ, U5 LM317LZ, U6 LM317LZ

Commit message: PCB: clemas con entrada hacia el borde, serigrafia, un solo puente; ERC/DRC sin errores
Co-Authored-By: Claude Opus 5.5 <noreply@anthropic.com>
Claude-Session: https://claude.ai/code/session_01WVk3oGwfQfGTmAT2PMp8oW
Parts:
- J1: Funcion Entrada de la fuente aislada de 36 VCC (pin 1 = 36V+, pin 2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 -> Entrada de la fuente aislada de 36 VCC (pin 2 = 36V+, pin 1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
- J3: Funcion Salida a las 3 flechas: pin 4 = +36V (ánodo común), 3 = F1-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 -> Salida a las 3 flechas: pin 1 = +36V (ánodo común), 2 = F1-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
- J4: Funcion Salida opcional CENTROS: pin 1 = retorno conmutado (-), pin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 -> Salida opcional CENTROS: pin 2 = retorno conmutado (-), pin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
- J5: Funcion Salida fija opcional FLORES (pin 1 = GND, pin 2 = +), resis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 -> Salida fija opcional FLORES (pin 1 = +, pin 2 = GND), resis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
- J6: Funcion Salida fija opcional BAÑOS (pin 1 = GND, pin 2 = +), resist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 -> Salida fija opcional BAÑOS (pin 1 = +, pin 2 = GND), resist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
- W1: footprint ControladorFlechas:Puente_Alambre_P15.24mm -> ControladorFlechas:Puente_Alambre_P7.62mm
Connections:
- net +36V: now also J3.1 (Pin_1); no longer J3.4 (Pin_4)
- net CENT_D: now also J4.2 (Pin_2); no longer J4.1 (Pin_1)
- net F1N: now also J3.2 (Pin_2); no longer J3.3 (Pin_3)
- net F2N: now also J3.3 (Pin_3); no longer J3.2 (Pin_2)
- net F3N: now also J3.4 (Pin_4); no longer J3.1 (Pin_1)
- net GND: now also J1.1 (Pin_1), J4.1 (Pin_1), J5.2 (Pin_2), J6.2 (Pin_2); no longer J1.2 (Pin_2), J4.2 (Pin_2), J5.1 (Pin_1), J6.1 (Pin_1)
- net VIN: now also J1.2 (Pin_2), J2.1 (Pin_1); no longer J1.1 (Pin_1), J2.2 (Pin_2)
- net VSW: now also J2.2 (Pin_2); no longer J2.1 (Pin_1)
- net V_BANO: now also J6.1 (Pin_1); no longer J6.2 (Pin_2)
- net V_FLOR: now also J5.1 (Pin_1); no longer J5.2 (Pin_2)
