File: hardware/flechas-127v/kicad/Flechas127.kicad_pcb (KiCad board)
At the start: 2 copper layers, 50 x 60 mm, 23 parts, among them J1 127 VCA, J2 FLECHAS, U1 NE555P, U2 CD4017BE

Commit message: Flechas 127 V: puentes W1/W2 del lado del cobre, pads sin agujero
Los dos puentes pasan a ser pads SMD en B.Cu (cable forrado soldado por abajo),
asi no se perforan 4 barrenos. ERC/DRC 0 con paridad; PDFs regenerados.

Co-Authored-By: Claude Opus 5.5 <noreply@anthropic.com>
Claude-Session: https://claude.ai/code/session_01WVk3oGwfQfGTmAT2PMp8oW
Parts:
- W1: footprint Flechas127:Puente_Alambre_P7.62mm -> Flechas127:Puente_Abajo_P7.62mm
- W2: footprint Flechas127:Puente_Alambre_P10.16mm -> Flechas127:Puente_Abajo_P10.16mm
Other:
- board text added: "W1 W2: CABLE FORRADO DEL LADO DEL COBRE"
- board text removed: "W1 W2: CABLE FORRADO"
