File: hardware/flechas-127v/kicad/Flechas127.kicad_sch (KiCad schematic)
At the start: 23 parts, among them J1 127 VCA, J2 FLECHAS, U1 NE555P, U2 CD4017BE

Commit message: Flechas 127 V: puentes W1/W2 del lado del cobre, pads sin agujero
Los dos puentes pasan a ser pads SMD en B.Cu (cable forrado soldado por abajo),
asi no se perforan 4 barrenos. ERC/DRC 0 con paridad; PDFs regenerados.

Co-Authored-By: Claude Opus 5.5 <noreply@anthropic.com>
Claude-Session: https://claude.ai/code/session_01WVk3oGwfQfGTmAT2PMp8oW
Parts:
- W1: footprint Flechas127:Puente_Alambre_P7.62mm -> Flechas127:Puente_Abajo_P7.62mm; Funcion Puente de alambre (lado componentes) que une CLK con CLK_W1 -> Puente de cable forrado del lado del cobre (sin agujero) qu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
- W2: footprint Flechas127:Puente_Alambre_P10.16mm -> Flechas127:Puente_Abajo_P10.16mm; Funcion Puente de alambre (lado componentes) que une V12 con V12_W2 -> Puente de cable forrado del lado del cobre (sin agujero) qu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
Changed lines of the file:
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@@
 			)
 		)
-		(property "Footprint" "Flechas127:Puente_Alambre_P7.62mm"
+		(property "Footprint" "Flechas127:Puente_Abajo_P7.62mm"
 			(at 40.64 127 0)
 			(hide yes)
@@
 			)
 		)
-		(property "Description" "Puente de alambre (lado componentes) que une CLK con CLK_W1"
+		(property "Description" "Puente de cable forrado del lado del cobre (sin agujero) que une CLK con CLK_W1"
 			(at 40.64 127 0)
 			(hide yes)
@@
 			)
 		)
-		(property "Funcion" "Puente de alambre (lado componentes) que une CLK con CLK_W1"
+		(property "Funcion" "Puente de cable forrado del lado del cobre (sin agujero) que une CLK con CLK_W1"
 			(at 40.64 127 0)
 			(hide yes)
@@
 			)
 		)
-		(property "Footprint" "Flechas127:Puente_Alambre_P10.16mm"
+		(property "Footprint" "Flechas127:Puente_Abajo_P10.16mm"
 			(at 71.12 127 0)
 			(hide yes)
@@
 			)
 		)
-		(property "Description" "Puente de alambre (lado componentes) que une V12 con V12_W2"
+		(property "Description" "Puente de cable forrado del lado del cobre (sin agujero) que une V12 con V12_W2"
 			(at 71.12 127 0)
 			(hide yes)
@@
 			)
 		)
-		(property "Funcion" "Puente de alambre (lado componentes) que une V12 con V12_W2"
+		(property "Funcion" "Puente de cable forrado del lado del cobre (sin agujero) que une V12 con V12_W2"
 			(at 71.12 127 0)
 			(hide yes)
