File: hardware/base12v/kicad/Base12V.kicad_sch (KiCad schematic)
At the start: 18 parts, among them J1 ENTRADA 12V, J2 SALIDAS, J3 HC-05, J4 MODO, Q1 IRLZ44N, Q2 IRLZ44N, Q3 IRLZ44N

Commit message: Base board v1.1: M3 mounting holes, security enclosure, 3D models, JLCPCB package, roadmap
- Board grows to 60 x 72 mm with 4 M3 holes; ERC/DRC 0 with schematic parity.
- Component 3D models (KiCad 9.0.0 STEP + simple Arduino Nano VRML).
- Printable tamper-proof enclosure (gen/caja.py -> STL) with PG7 glands,
  security-screw lid and warranty-seal recess, plus a 1:1 template for metal boxes.
- Gerber zip ready for JLCPCB/PCBWay.
- HOJA_DE_RUTA.md: phases from home-made board to factory assembly.

Co-Authored-By: Claude Opus 5.5 <noreply@anthropic.com>
Claude-Session: https://claude.ai/code/session_01WVk3oGwfQfGTmAT2PMp8oW
Other:
- company: PCB 50 x 60 mm, una cara, THT, transferencia de toner -> PCB 60 x 72 mm, una cara, THT, 4 barrenos M3, transferencia de toner
Changed lines of the file:
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@@
 		(date "2026-10-01")
 		(rev "1.0")
-		(company "PCB 50 x 60 mm, una cara, THT, transferencia de toner")
+		(company "PCB 60 x 72 mm, una cara, THT, 4 barrenos M3, transferencia de toner")
 		(comment 1 "Bajo voltaje aislado: eliminador/fuente switching de 12 V regulada")
 		(comment 2 "Canales: tira 12 V, LED 5 mm con resistencia o tira RGB anodo comun")
