File: hardware/ap1-ensamble/AP1_Ensamble.kicad_pcb (KiCad board)
At the start: 2 copper layers, 88 x 56 mm, 69 parts, among them J1 ENTRADA 12-24V, J3 +V SALIDA, J4 CANALES, J5 FOCOS CC, J6 AUX 12V, J7 PROGRAMADOR, Q1 BSC028N06LS3, Q2 BSC028N06LS3, Q3 BSC028N06LS3, Q4 BSC028N06LS3, Q5 AO3400A, U1 INA238, U2 LMR16006XDDC, U3 UCC27524D, U4 UCC27524D, U6 AL8860MP, U7 AL8860MP, U8 TMP1075D, U9 AT24CS02

Commit message: Gabinete imprimible para el conjunto AP-1, revisado contra el modelo 3D real
- ap1-gabinete/gen/caja.py: caja de 95 x 78 x 38 mm con 3 postes M3, 4 PG7 al
  frente, ventana USB-C atrás, tapa con ventana IR, tubos de luz, BOOT/RESET
  y textos grabados, columnas de tornillos por fuera de la placa y orejas.
- Carga AP1_Ensamble.step y falla si alguna pieza toca la caja: 0 choques,
  2.5 mm de holgura a la tapa.
- Plantilla 1:1 para caja comprada de plástico.
- ap1-ensamble: modelos del programador y del conjunto actualizados.

Co-Authored-By: Claude Opus 5.5 <noreply@anthropic.com>
Claude-Session: https://claude.ai/code/session_01WVk3oGwfQfGTmAT2PMp8oW
Parts:
- added D8: 1N4148WS, Diode_SMD:D_SOD-323, F.Cu at (151.6, 120.6)
- added D9: 1N4148WS, Diode_SMD:D_SOD-323, F.Cu at (165.4, 120.6)
- D1: value SMBJ33A -> SMBJ26A
- U9: value AT24CS02 -> M24C02-WMN6TP; footprint Package_TO_SOT_SMD:SOT-23-5 -> Package_SO:SOIC-8_3.9x4.9mm_P1.27mm
- moved U9 2.50 mm to (153.0, 109.5)
Connections:
- U3 pad 1: unconnected-(U3-ENA-Pad1) -> /EN12
- U3 pad 8: unconnected-(U3-ENB-Pad8) -> /EN12
- U4 pad 1: unconnected-(U4-ENA-Pad1) -> /EN34
- U4 pad 8: unconnected-(U4-ENB-Pad8) -> /EN34
- U9 pad 1: /SCL -> /GND
- U9 pad 3: /SDA -> /GND
- U9 pad 4: /3V3 -> /GND
- U9 pad 5: /GND -> /SDA
Routing:
- net /GND: track 248.4 -> 101.9 mm, vias 51 -> 93
- net /3V3: track 60.0 -> 80.7 mm, vias 2 -> 1
- net /LEDK1: track 45.6 -> 35.9 mm
- net /ALERT: track 32.4 -> 40.9 mm
- net /EN34: track 0.00 -> 8.10 mm
- net /EN12: track 0.00 -> 7.79 mm
- net /AUX: track 47.4 -> 55.2 mm, vias 0 -> 1
- net /PWM1: track 17.4 -> 24.8 mm, vias 2 -> 1
- net /PWM3: track 24.2 -> 18.8 mm
- net /LEDA1: track 42.3 -> 38.4 mm
- net /LEDK2: track 25.4 -> 21.7 mm
- net /SWC1: track 15.0 -> 18.4 mm
- net /VCC: track 74.2 -> 71.5 mm, vias 4 -> 3
- net /SDA: track 43.3 -> 41.2 mm, vias 1 -> 0
- net /SWC2: track 17.4 -> 19.0 mm, vias 2 -> 0
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- added copper zone on In1.Cu, net /GND
- added copper zone on In2.Cu, net /GND
Other:
- copper layers 2 -> 4
