File: hardware/ap02/kicad/AP02.kicad_pcb (KiCad board)
At the start: 2 copper layers, 90 x 70 mm, 71 parts, among them J1 ENTRADA 12-24V, J2 USB-C, J3 +V SALIDA, J4 CANALES, J5 FOCOS, J6 EXPANSION, K1 SRD-12VDC-SL-C, Q1 BSC028N06LS3, Q2 BSC028N06LS3, Q3 BSC028N06LS3, Q4 BSC028N06LS3, Q5 AO3400A, SW1 MODO / BOOT, SW2 RESET, U1 AP63203WU, U2 AP63200WU, U3 UCC27524D, U4 UCC27524D, U5 ESP32-C3-WROOM-02, U6 USBLC6-2SC6

Commit message: AP-0.2 rev B: regulador de 60 V, medidor de potencia, protecciones y planos de 20 A
Placa:
- Buck de 12 V LMR16006 (60 V) en lugar de AP63200 (32 V); la logica toma de los 12 V
- INA238 (85 V) con shunt Kelvin de 1 mOhm: V, A, W, kWh y alerta por sobrecorriente
- TMP1075 junto a drivers y MOSFET; alertas a IO20
- Planos de entrada de 7.3 y 11 mm (antes 3.8/4.4 mm); TVS despues del fusible
- Capacitores de 50 V; 6 puntos de prueba de fabrica
- Areas prohibidas durante el ruteo para que Freerouting no parta los planos;
  ruteo en 3 pasadas, en un hilo y reproducible (gen/rutear.sh)
- ERC/DRC sin errores ni advertencias, 0 sin conectar, paridad con el esquema

Programa 1.1:
- Lectura de INA238/TMP1075, kWh guardados, corte por sobrecorriente,
  sobrevoltaje y temperatura con reintento, menos brillo desde 70 C
- PWM desfasado entre canales y arranque suave de 0.6 s
- App: tarjeta de consumo, aviso de proteccion y limite de corriente

Co-Authored-By: Claude Opus 5.5 <noreply@anthropic.com>
Claude-Session: https://claude.ai/code/session_01WVk3oGwfQfGTmAT2PMp8oW
Parts:
- added C17: 100nF, Capacitor_SMD:C_0603_1608Metric, F.Cu at (104.0, 133.5)
- added C18: 100nF, Capacitor_SMD:C_0603_1608Metric, F.Cu at (144.0, 132.0)
- added R15: 10k, Resistor_SMD:R_0603_1608Metric, F.Cu at (144.0, 130.3)
- added RS1: 1mR 2512 Kelvin, Resistor_SMD:R_Shunt_Vishay_WSK2512_6332Metric_T1.19mm, F.Cu at (110.9, 140.8)
- added TP1: VIN, TestPoint:TestPoint_Pad_D1.5mm, F.Cu at (105.5, 147.5)
- added TP2: 12V, TestPoint:TestPoint_Pad_D1.5mm, F.Cu at (138.5, 126.0)
- added TP3: 3V3, TestPoint:TestPoint_Pad_D1.5mm, F.Cu at (154.0, 123.5)
- added TP4: GND, TestPoint:TestPoint_Pad_D1.5mm, F.Cu at (154.0, 126.3)
- added TP5: TXD, TestPoint:TestPoint_Pad_D1.5mm, F.Cu at (156.6, 123.5)
- added TP6: EN, TestPoint:TestPoint_Pad_D1.5mm, F.Cu at (156.6, 126.3)
- added U7: INA238, Package_SO:VSSOP-10_3x3mm_P0.5mm, F.Cu at (106.0, 136.3)
- added U8: TMP1075D, Package_SO:SOIC-8_3.9x4.9mm_P1.27mm, F.Cu at (144.0, 137.0)
- C1, C2: value 470uF 35V -> 330uF 50V
- L2: value 10uH -> 47uH
- RF1: value 140k -> 150k
- U2: value AP63200WU -> LMR16006XDDC; footprint Package_TO_SOT_SMD:TSOT-23-6 -> Package_TO_SOT_SMD:SOT-23-6
- moved C3 28.2 mm to (106.5, 151.0)
- moved D1 17.0 mm to (120.5, 132.6)
- moved C1 2.50 mm to (110.0, 127.0), turned to 180 degrees
- moved C2 1.20 mm to (110.0, 112.8), turned to 180 degrees
Connections:
- C1 pad 1: /VIN -> /VFUS
- C2 pad 1: /VIN -> /VFUS
- C9 pad 1: /VIN -> /VFUS
- D1 pad 1: /VIN -> /VFUS
- D2 pad 2: /VIN -> /V12G
- F1 pad 2: /VIN -> /VFUS
- RG0 pad 1: /VIN -> /VFUS
- U2 pad 1: /FB2 -> /BST2
- U2 pad 2: /VIN -> /GND
- U2 pad 3: /VIN -> /FB2
- U2 pad 4: /GND -> /VFUS
- U2 pad 5: /SW2 -> /VFUS
- U2 pad 6: /BST2 -> /SW2
- U5 pad 11: unconnected-(U5-IO20/RXD-Pad11) -> /ALERT
- U5 pad 12: unconnected-(U5-IO21/TXD-Pad12) -> /TXD
Routing:
- net /SDA: track 12.1 -> 116.9 mm, vias 0 -> 3
- net /ALERT: track 0.00 -> 87.6 mm, vias 0 -> 3
- net /SCL: track 38.9 -> 113.8 mm, vias 1 -> 4
- net /3V3: track 103.3 -> 175.1 mm, vias 2 -> 1
- net /GND: track 286.2 -> 351.2 mm, vias 54 -> 58
- net /VIN: track 62.2 -> 0.00 mm, vias 2 -> 0
- net /TXD: track 0.00 -> 22.3 mm, vias 0 -> 2
- net /VFUS: track 0.00 -> 20.1 mm
- net /V12G: track 97.3 -> 115.9 mm, vias 3 -> 5
- net /ISN: track 0.00 -> 15.9 mm, vias 0 -> 2
- net /PWM4: track 39.4 -> 24.9 mm
- net /ISP: track 0.00 -> 13.5 mm, vias 0 -> 2
- net /PWM2: track 44.5 -> 33.6 mm
- net /PWM1: track 41.7 -> 33.2 mm
- net /EN: track 41.6 -> 49.1 mm, vias 2 -> 3
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- added copper zone on F.Cu, net /VFUS
Other:
- board text added: "12-24V 20A, mide y protege"
- board text added: "8 A max por canal - 20 A total"
- board text added: "LetreroLab AP-0.2 rev B"
- board text removed: "12-24V 20A max"
- board text removed: "8A/canal"
- board text removed: "LetreroLab AP-0.2"

Commit message: AP-1: base universal + programador que se enclava; AP-0.2 rev C
AP-1 BASE universal (88 x 56 mm, 2 oz):
- Entrada 12-24 V 20 A con fusible mini de auto, polaridad sin pérdidas,
  TVS y medidor INA238 con shunt Kelvin de 1 mOhm
- 4 canales de 8 A, 2 canales de corriente constante AL8860 (focos, 1 A,
  salidas flotantes con fusible propio), salida AUX 12 V para relevador o
  contactor externo (la red no entra a la placa) o ventilador
- Fuente LMR16006 60 V -> 12 V con su diodo, TMP1075, memoria AT24CS02
  con número de serie de fábrica, zócalo 2x8 para el programador
- Zona sin cobre bajo la antena y franja de retorno sin pistas en la capa
  inferior; áreas prohibidas al rutear sobre los planos de potencia

AP-1 PROGRAMADOR (52 x 42 mm): ESP32-C3, USB-C, AP63203, botones,
LED OK y LED de FALLA por hardware, IR, Qwiic, conector macho abajo.
Las 16 patas y el tornillo coinciden con la base (verificado).

Firmware AP-1: diagnóstico de salidas con el medidor de la base (5 % para
detectar cortos, luego 100 %), aprender consumo normal y aviso de
desviación, focos CC, AUX/ventilador, datos de la base, OLED y BH1750.

AP-0.2 rev C: diodo de rueda libre del LMR16006 (faltaba en la rev B) y
pull-down en los 4 PWM para que no enciendan al arrancar el ESP32.

Herramientas: tools/placa.py (librería de generación), rutear.sh,
salidas.py, modelos_locales.py; modelo 3D del conjunto en ap1-ensamble.
Todas las placas: ERC 0, DRC 0, 0 sin conectar, 0 diferencias.

Co-Authored-By: Claude Opus 5.5 <noreply@anthropic.com>
Claude-Session: https://claude.ai/code/session_01WVk3oGwfQfGTmAT2PMp8oW
Parts:
- added D6: SS210, Diode_SMD:D_SMA, F.Cu at (130.5, 127.0)
- added RPD1: 10k, Resistor_SMD:R_0603_1608Metric, F.Cu at (155.6, 115.0)
- added RPD2: 10k, Resistor_SMD:R_0603_1608Metric, F.Cu at (155.6, 116.8)
- added RPD3: 10k, Resistor_SMD:R_0603_1608Metric, F.Cu at (155.6, 118.6)
- added RPD4: 10k, Resistor_SMD:R_0603_1608Metric, F.Cu at (155.6, 120.4)
Routing:
- net /PWM1: track 33.2 -> 52.1 mm
- net /SCL: track 113.8 -> 95.7 mm
- net /EN: track 49.1 -> 64.9 mm
- net /TXD: track 22.3 -> 37.8 mm
- net /PWM2: track 33.6 -> 47.2 mm, vias 2 -> 3
- net /SDA: track 116.9 -> 103.6 mm, vias 3 -> 4
- net /PWM3: track 23.3 -> 30.3 mm, vias 2 -> 3
- net /V12G: track 115.9 -> 121.0 mm, vias 5 -> 6
- net /USB_DP: track 28.1 -> 23.5 mm
- net /ALERT: track 87.6 -> 83.3 mm, vias 3 -> 5
- net /SW2: track 11.2 -> 15.5 mm
- net /PWM4: track 24.9 -> 28.7 mm
- net /3V3: track 175.1 -> 171.7 mm, vias 1 -> 3
- net /GND: track 351.2 -> 348.0 mm, vias 58 -> 66
- net /GO1: track 14.2 -> 11.2 mm, vias 2 -> 0
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Other:
- board text added: "LetreroLab AP-0.2 rev C"
- board text removed: "LetreroLab AP-0.2 rev B"

Commit message: Pedido más económico en JLCPCB: menos piezas Extended y BOM solo SMD
- Base: memoria AT24CS02 -> M24C02 (Preferred). El programa crea el número
  de serie (128 bits al azar con la MAC del programador) si la memoria no trae.
- Programador y AP-0.2: botones TL3342 -> TS-1187A (Basic, misma huella).
  En la AP-0.2 se cambió la huella sin volver a rutear: DRC 0.
- Base: rutas fijas para SWC1/SWC2 y CC2 igual que CC1 (el canal 2 es
  copia del 1, 12.5 mm abajo). Ruteo estable: ERC 0, DRC 0, 0 sin conectar.
- salidas.py: BOM/CPL '_solo_SMD' para soldar a mano clemas y conectores,
  resumen con cargo por código LCSC distinto y costo de piezas Basic.
- jlcpcb.py: piezas reconocidas por huella (botones con valor de etiqueta).
- Cargo de montaje por pedido: base+programador de ~93 a ~84 USD, o ~54 USD
  en el pedido solo SMD.

Co-Authored-By: Claude Opus 5.5 <noreply@anthropic.com>
Claude-Session: https://claude.ai/code/session_01WVk3oGwfQfGTmAT2PMp8oW
Parts:
- SW1, SW2: footprint Button_Switch_SMD:SW_SPST_TL3342 -> Button_Switch_SMD:SW_Push_1P1T_XKB_TS-1187A

Commit message: AP-0.2 rev D: corte de MOSFET por hardware, botones Basic y Home Assistant
- D7/D8 (1N4148WS) llevan ALERTA (INA238/TMP1075) a los EN de los UCC27524:
  los MOSFET se apagan sin depender del programa. Ruteada otra vez:
  ERC 0, DRC 0, 0 sin conectar, 0 diferencias. Serigrafía rev D.
- Programa fw 1.2: alerta del INA238 en menos de 1 ms, descubrimiento MQTT
  de Home Assistant (luz, relevador y sensores), varias órdenes por mensaje.
- Salidas regeneradas con BOM/CPL solo SMD (cargo ~60 -> ~39 USD).

Co-Authored-By: Claude Opus 5.5 <noreply@anthropic.com>
Claude-Session: https://claude.ai/code/session_01WVk3oGwfQfGTmAT2PMp8oW
Parts:
- added D7: 1N4148WS, Diode_SMD:D_SOD-323, F.Cu at (140.2, 129.8)
- added D8: 1N4148WS, Diode_SMD:D_SOD-323, F.Cu at (148.0, 129.8)
Connections:
- U3 pad 1: unconnected-(U3-ENA-Pad1) -> /EN12
- U3 pad 8: unconnected-(U3-ENB-Pad8) -> /EN12
- U4 pad 1: unconnected-(U4-ENA-Pad1) -> /EN34
- U4 pad 8: unconnected-(U4-ENB-Pad8) -> /EN34
Routing:
- net /ALERT: track 83.3 -> 108.5 mm
- net /TXD: track 37.8 -> 21.7 mm
- net /EN: track 64.9 -> 49.4 mm
- net /GND: track 348.0 -> 362.2 mm, vias 66 -> 60
- net /SCL: track 95.7 -> 108.2 mm, vias 4 -> 6
- net /EN12: track 0.00 -> 11.0 mm
- net /EN34: track 0.00 -> 10.2 mm
- net /SDA: track 103.6 -> 113.3 mm
- net /BOOT: track 52.0 -> 59.6 mm, vias 0 -> 2
- net /RLYG: track 49.4 -> 42.8 mm
- net /VLOG: track 40.8 -> 34.2 mm, vias 0 -> 2
- net /PWM2: track 47.2 -> 40.9 mm
- net /PWM1: track 52.1 -> 47.3 mm
- net /LDR: track 28.2 -> 25.8 mm
- net /PWM3: track 30.3 -> 32.5 mm
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Other:
- board text added: "LetreroLab AP-0.2 rev D"
- board text removed: "LetreroLab AP-0.2 rev C"

Commit message: Listo para JLCPCB: códigos LCSC, reglas de fabricación y carpeta de pedido
- Códigos LCSC verificados para todas las piezas SMD (INA238, LMR16006,
  UCC27524, AL8860, TMP1075, MOSFET, bobinas, capacitor, fusible, módulo,
  conectores) en tools/jlcpcb.py; piezas reconocidas por huella.
- Shunt: el WSK2512 de 4 terminales se agotó en LCSC; base y AP-0.2 usan un
  HoJLR2512 1 mOhm 2 W (C2924520) con huella propia 'net tie' que conserva
  el sensado Kelvin (tools/huellas/LetreroLab.pretty).
- ESP32-C3-WROOM-02: huella propia con 4 vías de 0.3 mm en lugar de 12 de
  0.2 mm (proceso estándar de JLCPCB). Textos de serigrafía de 0.8 mm o más.
- IND: fusible de 3 A (el mismo de la base).
- AP-0.2 ruteada otra vez con el nuevo shunt.
- Las 4 placas: ERC 0, DRC 0, 0 sin conectar, 0 diferencias y 0 problemas
  con las reglas de fabricación de JLCPCB.
- PEDIDO_JLCPCB/ (+ .zip) con Gerber, BOM y CPL completos o solo SMD por
  placa, y PEDIDO_JLCPCB.md con las opciones exactas del pedido.

Co-Authored-By: Claude Opus 5.5 <noreply@anthropic.com>
Claude-Session: https://claude.ai/code/session_01WVk3oGwfQfGTmAT2PMp8oW
Parts:
- RS1: value 1mR 2512 Kelvin -> 1mR 2512 2W; footprint Resistor_SMD:R_Shunt_Vishay_WSK2512_6332Metric_T1.19mm -> LetreroLab:R_2512_Kelvin_NetTie
- U5: footprint RF_Module:ESP32-C3-WROOM-02 -> LetreroLab:ESP32-C3-WROOM-02_JLC
Routing:
- net /V12G: track 120.1 -> 135.7 mm
- net /SDA: track 113.3 -> 102.2 mm, vias 4 -> 3
- net /3V3: track 171.8 -> 181.0 mm, vias 3 -> 6
- net /RLYG: track 42.8 -> 50.2 mm
- net /ALERT: track 108.5 -> 101.5 mm, vias 5 -> 7
- net /USB_DN: track 24.7 -> 31.4 mm, vias 3 -> 2
- net /SW1: track 13.9 -> 7.63 mm, vias 2 -> 0
- net /PWM2: track 40.9 -> 46.9 mm
- net /BOOT: track 59.6 -> 65.1 mm, vias 2 -> 3
- net /EN: track 49.4 -> 44.5 mm, vias 3 -> 4
- net /VBUS: track 59.7 -> 55.0 mm
- net /LED: track 25.1 -> 29.7 mm
- net /FB2: track 12.7 -> 8.57 mm
- net /LDR: track 25.8 -> 29.8 mm, vias 1 -> 0
- net /GREV: track 17.1 -> 19.9 mm
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