File: hardware/ap02/kicad/AP02.kicad_sch (KiCad schematic)
At the start: 68 parts, among them J1 ENTRADA 12-24V, J2 USB-C, J3 +V SALIDA, J4 CANALES, J5 FOCOS, J6 EXPANSION, K1 SRD-12VDC-SL-C, Q1 BSC028N06LS3, Q2 BSC028N06LS3, Q3 BSC028N06LS3, Q4 BSC028N06LS3, Q5 AO3400A, SW1 MODO / BOOT, SW2 RESET, U1 AP63203WU, U2 AP63200WU, U3 UCC27524D, U4 UCC27524D, U5 ESP32-C3-WROOM-02, U6 USBLC6-2SC6

Commit message: AP-0.2 rev B: regulador de 60 V, medidor de potencia, protecciones y planos de 20 A
Placa:
- Buck de 12 V LMR16006 (60 V) en lugar de AP63200 (32 V); la logica toma de los 12 V
- INA238 (85 V) con shunt Kelvin de 1 mOhm: V, A, W, kWh y alerta por sobrecorriente
- TMP1075 junto a drivers y MOSFET; alertas a IO20
- Planos de entrada de 7.3 y 11 mm (antes 3.8/4.4 mm); TVS despues del fusible
- Capacitores de 50 V; 6 puntos de prueba de fabrica
- Areas prohibidas durante el ruteo para que Freerouting no parta los planos;
  ruteo en 3 pasadas, en un hilo y reproducible (gen/rutear.sh)
- ERC/DRC sin errores ni advertencias, 0 sin conectar, paridad con el esquema

Programa 1.1:
- Lectura de INA238/TMP1075, kWh guardados, corte por sobrecorriente,
  sobrevoltaje y temperatura con reintento, menos brillo desde 70 C
- PWM desfasado entre canales y arranque suave de 0.6 s
- App: tarjeta de consumo, aviso de proteccion y limite de corriente

Co-Authored-By: Claude Opus 5.5 <noreply@anthropic.com>
Claude-Session: https://claude.ai/code/session_01WVk3oGwfQfGTmAT2PMp8oW
Parts:
- added C17, C18: 100nF, Capacitor_SMD:C_0603_1608Metric, symbol Device:C
- added R15: 10k, Resistor_SMD:R_0603_1608Metric, symbol Device:R
- added RS1: 1mR 2512 Kelvin, Resistor_SMD:R_Shunt_Vishay_WSK2512_6332Metric_T1.19mm, symbol Device:R_Shunt
- added TP1: VIN, TestPoint:TestPoint_Pad_D1.5mm, symbol Connector:TestPoint
- added TP2: 12V, TestPoint:TestPoint_Pad_D1.5mm, symbol Connector:TestPoint
- added TP3: 3V3, TestPoint:TestPoint_Pad_D1.5mm, symbol Connector:TestPoint
- added TP4: GND, TestPoint:TestPoint_Pad_D1.5mm, symbol Connector:TestPoint
- added TP5: TXD, TestPoint:TestPoint_Pad_D1.5mm, symbol Connector:TestPoint
- added TP6: EN, TestPoint:TestPoint_Pad_D1.5mm, symbol Connector:TestPoint
- added U7: INA238, Package_SO:VSSOP-10_3x3mm_P0.5mm, symbol Sensor_Energy:INA238
- added U8: TMP1075D, Package_SO:SOIC-8_3.9x4.9mm_P1.27mm, symbol Sensor_Temperature:TMP1075D
- C1, C2: value 470uF 35V -> 330uF 50V; Funcion Filtro de entrada -> Filtro de entrada (50 V, 105 C, bajo ESR, larga vida)
- C3: Funcion Desacoplo cerca de los MOSFET -> Desacoplo de la salida +V junto a J3 (lazo corto con las ti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
- D1: Funcion Supresor de picos -> Supresor de picos (despues del fusible: una falla sostenida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
- D2: Funcion Alimenta la logica desde VIN -> Alimenta la logica desde los 12 V internos
- L2: value 10uH -> 47uH
- RF1: value 140k -> 150k; Funcion Divisor de 12 V (0.8 V x 15) -> Divisor: 0.765 V x 16 = 12.2 V
- U1: Funcion Buck 3.3 V 2 A (3.8-32 V) -> Buck 3.3 V 2 A (entrada 5-12 V: USB o 12 V internos)
- U2: value AP63200WU -> LMR16006XDDC; footprint Package_TO_SOT_SMD:TSOT-23-6 -> Package_TO_SOT_SMD:SOT-23-6; symbol Regulator_Switching:AP63200WU -> Regulator_Switching:LMR16006YQ; Funcion Buck 12 V (drivers y relevador) -> Buck 12 V de 60 V / 0.6 A, 700 kHz (drivers, relevador y lo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
Connections:
- net 3V3: now also C17.1, C18.1, R15.1, TP3.1, U7.6 (VS), U8.8 (V+)
- net BST2: now also U2.1 (CB); no longer U2.6 (BST)
- net EN: now also TP6.1
- net FB2: now also U2.3 (FB); no longer U2.1 (FB)
- net GND: now also U2.2 (GND), C17.2, C18.2, TP4.1, U7.1 (A1), U7.2 (A0), U7.7 (GND), U8.4 (GND), U8.5 (A2), U8.6 (A1), U8.7 (A0); no longer U2.4 (GND)
- net SCL: now also U7.5 (SCL), U8.2 (SCL)
- net SDA: now also U7.4 (SDA), U8.1 (SDA)
- net SW2: now also U2.6 (SW); no longer U2.5 (SW)
- net V12G: now also D2.2 (A), TP2.1
- net VIN: now also RS1.1, TP1.1; no longer C1.1, C2.1, C9.1, D1.1 (A1), D2.2 (A), F1.2, RG0.1, U2.2 (EN), U2.3 (IN)
- net ALERT: now reaches U5.11 (IO20/RXD)
- net ALERT: now also R15.2, U7.3 (~{Alert}), U8.3 (ALERT)
- net TXD: now reaches U5.12 (IO21/TXD)
- net TXD: now also TP5.1
- new net ISN: RS1.2, U7.8 (Vbus), U7.9 (Vin-)
- new net ISP: RS1.3, U7.10 (Vin+)
- new net VFUS: C1.1, C2.1, C9.1, D1.1 (A1), F1.2, RG0.1, RS1.4, U2.4 (~{SHDN}), U2.5 (VIN)
- no-connect marks 9 -> 7
Other:
- note added: "LetreroLab AP-0.2: entrada 12-24 V / 20 A, 4 canales de 8 A, ESP32-C3 Wi-Fi, relevador 10 A. PWM1-4 = IO4-IO7, relevador = IO1, LED = IO10, IR = IO3, LDR = IO0, SDA/SCL = IO2/IO8, MODO = IO9, ALERTA (INA238 0x40 + TMP1075 0x48) = IO20, TXD de prueba = IO21. Shunt 1 mOhm Kelvin."
- note removed: "LetreroLab AP-0.2: entrada 12-24 V / 20 A, 4 canales de 8 A, ESP32-C3 Wi-Fi, relevador 10 A. PWM1-4 = IO4-IO7, relevador = IO1, LED = IO10, IR = IO3, LDR = IO0, SDA/SCL = IO2/IO8, MODO = IO9."
- moved on the sheet: C1, C10, C11, C12, C13, C14, C15, C16, C2, C3, C4, C5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

Commit message: AP-1: base universal + programador que se enclava; AP-0.2 rev C
AP-1 BASE universal (88 x 56 mm, 2 oz):
- Entrada 12-24 V 20 A con fusible mini de auto, polaridad sin pérdidas,
  TVS y medidor INA238 con shunt Kelvin de 1 mOhm
- 4 canales de 8 A, 2 canales de corriente constante AL8860 (focos, 1 A,
  salidas flotantes con fusible propio), salida AUX 12 V para relevador o
  contactor externo (la red no entra a la placa) o ventilador
- Fuente LMR16006 60 V -> 12 V con su diodo, TMP1075, memoria AT24CS02
  con número de serie de fábrica, zócalo 2x8 para el programador
- Zona sin cobre bajo la antena y franja de retorno sin pistas en la capa
  inferior; áreas prohibidas al rutear sobre los planos de potencia

AP-1 PROGRAMADOR (52 x 42 mm): ESP32-C3, USB-C, AP63203, botones,
LED OK y LED de FALLA por hardware, IR, Qwiic, conector macho abajo.
Las 16 patas y el tornillo coinciden con la base (verificado).

Firmware AP-1: diagnóstico de salidas con el medidor de la base (5 % para
detectar cortos, luego 100 %), aprender consumo normal y aviso de
desviación, focos CC, AUX/ventilador, datos de la base, OLED y BH1750.

AP-0.2 rev C: diodo de rueda libre del LMR16006 (faltaba en la rev B) y
pull-down en los 4 PWM para que no enciendan al arrancar el ESP32.

Herramientas: tools/placa.py (librería de generación), rutear.sh,
salidas.py, modelos_locales.py; modelo 3D del conjunto en ap1-ensamble.
Todas las placas: ERC 0, DRC 0, 0 sin conectar, 0 diferencias.

Co-Authored-By: Claude Opus 5.5 <noreply@anthropic.com>
Claude-Session: https://claude.ai/code/session_01WVk3oGwfQfGTmAT2PMp8oW
Parts:
- added D6: SS210, Diode_SMD:D_SMA, symbol Device:D_Schottky
- added RPD1, RPD2, RPD3, RPD4: 10k, Resistor_SMD:R_0603_1608Metric, symbol Device:R
Connections:
- net GND: now also D6.2 (A), RPD1.2, RPD2.2, RPD3.2, RPD4.2
- net PWM1: now also RPD1.1
- net PWM2: now also RPD2.1
- net PWM3: now also RPD3.1
- net PWM4: now also RPD4.1
- net SW2: now also D6.1 (K)
Other:
- moved on the sheet: C10, C11, C12, C13, C14, C15, C16, C18, C8, C9, D4, D5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

Commit message: Pedido más económico en JLCPCB: menos piezas Extended y BOM solo SMD
- Base: memoria AT24CS02 -> M24C02 (Preferred). El programa crea el número
  de serie (128 bits al azar con la MAC del programador) si la memoria no trae.
- Programador y AP-0.2: botones TL3342 -> TS-1187A (Basic, misma huella).
  En la AP-0.2 se cambió la huella sin volver a rutear: DRC 0.
- Base: rutas fijas para SWC1/SWC2 y CC2 igual que CC1 (el canal 2 es
  copia del 1, 12.5 mm abajo). Ruteo estable: ERC 0, DRC 0, 0 sin conectar.
- salidas.py: BOM/CPL '_solo_SMD' para soldar a mano clemas y conectores,
  resumen con cargo por código LCSC distinto y costo de piezas Basic.
- jlcpcb.py: piezas reconocidas por huella (botones con valor de etiqueta).
- Cargo de montaje por pedido: base+programador de ~93 a ~84 USD, o ~54 USD
  en el pedido solo SMD.

Co-Authored-By: Claude Opus 5.5 <noreply@anthropic.com>
Claude-Session: https://claude.ai/code/session_01WVk3oGwfQfGTmAT2PMp8oW
Parts:
- SW1, SW2: footprint Button_Switch_SMD:SW_SPST_TL3342 -> Button_Switch_SMD:SW_Push_1P1T_XKB_TS-1187A
Changed lines of the file:
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@@
 			)
 		)
-		(property "Footprint" "Button_Switch_SMD:SW_SPST_TL3342"
+		(property "Footprint" "Button_Switch_SMD:SW_Push_1P1T_XKB_TS-1187A"
 			(at 73.66 307.34 0)
 			(hide yes)
@@
 			)
 		)
-		(property "Footprint" "Button_Switch_SMD:SW_SPST_TL3342"
+		(property "Footprint" "Button_Switch_SMD:SW_Push_1P1T_XKB_TS-1187A"
 			(at 116.84 307.34 0)
 			(hide yes)

Commit message: AP-0.2 rev D: corte de MOSFET por hardware, botones Basic y Home Assistant
- D7/D8 (1N4148WS) llevan ALERTA (INA238/TMP1075) a los EN de los UCC27524:
  los MOSFET se apagan sin depender del programa. Ruteada otra vez:
  ERC 0, DRC 0, 0 sin conectar, 0 diferencias. Serigrafía rev D.
- Programa fw 1.2: alerta del INA238 en menos de 1 ms, descubrimiento MQTT
  de Home Assistant (luz, relevador y sensores), varias órdenes por mensaje.
- Salidas regeneradas con BOM/CPL solo SMD (cargo ~60 -> ~39 USD).

Co-Authored-By: Claude Opus 5.5 <noreply@anthropic.com>
Claude-Session: https://claude.ai/code/session_01WVk3oGwfQfGTmAT2PMp8oW
Parts:
- added D7, D8: 1N4148WS, Diode_SMD:D_SOD-323, symbol Device:D
Connections:
- net ALERT: now also D7.1 (K), D8.1 (K)
- net EN34: now reaches U4.1 (ENA)
- net EN34: now also U4.8 (ENB), D8.2 (A)
- net EN12: now reaches U3.1 (ENA)
- net EN12: now also U3.8 (ENB), D7.2 (A)
- no-connect marks 7 -> 3
Other:
- moved on the sheet: C11, C12, C13, C14, C15, C16, C18, D4, D5, J2, J5, J6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

Commit message: Listo para JLCPCB: códigos LCSC, reglas de fabricación y carpeta de pedido
- Códigos LCSC verificados para todas las piezas SMD (INA238, LMR16006,
  UCC27524, AL8860, TMP1075, MOSFET, bobinas, capacitor, fusible, módulo,
  conectores) en tools/jlcpcb.py; piezas reconocidas por huella.
- Shunt: el WSK2512 de 4 terminales se agotó en LCSC; base y AP-0.2 usan un
  HoJLR2512 1 mOhm 2 W (C2924520) con huella propia 'net tie' que conserva
  el sensado Kelvin (tools/huellas/LetreroLab.pretty).
- ESP32-C3-WROOM-02: huella propia con 4 vías de 0.3 mm en lugar de 12 de
  0.2 mm (proceso estándar de JLCPCB). Textos de serigrafía de 0.8 mm o más.
- IND: fusible de 3 A (el mismo de la base).
- AP-0.2 ruteada otra vez con el nuevo shunt.
- Las 4 placas: ERC 0, DRC 0, 0 sin conectar, 0 diferencias y 0 problemas
  con las reglas de fabricación de JLCPCB.
- PEDIDO_JLCPCB/ (+ .zip) con Gerber, BOM y CPL completos o solo SMD por
  placa, y PEDIDO_JLCPCB.md con las opciones exactas del pedido.

Co-Authored-By: Claude Opus 5.5 <noreply@anthropic.com>
Claude-Session: https://claude.ai/code/session_01WVk3oGwfQfGTmAT2PMp8oW
Parts:
- RS1: value 1mR 2512 Kelvin -> 1mR 2512 2W; footprint Resistor_SMD:R_Shunt_Vishay_WSK2512_6332Metric_T1.19mm -> LetreroLab:R_2512_Kelvin_NetTie; Funcion Shunt de 1 mOhm (4 terminales) para medir la corriente total -> Shunt de 1 mOhm 2 W (HoJLR2512, C2924520, en existencia) co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
- U5: footprint RF_Module:ESP32-C3-WROOM-02 -> LetreroLab:ESP32-C3-WROOM-02_JLC
Changed lines of the file:
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@@
 			)
 		)
-		(property "Value" "1mR 2512 Kelvin"
+		(property "Value" "1mR 2512 2W"
 			(at 131.38 42.24 0)
 			(effects
@@
 			)
 		)
-		(property "Footprint" "Resistor_SMD:R_Shunt_Vishay_WSK2512_6332Metric_T1.19mm"
+		(property "Footprint" "LetreroLab:R_2512_Kelvin_NetTie"
 			(at 116.84 40.64 0)
 			(hide yes)
@@
 			)
 		)
-		(property "Description" "Shunt de 1 mOhm (4 terminales) para medir la corriente total"
+		(property "Description" "Shunt de 1 mOhm 2 W (HoJLR2512, C2924520, en existencia) con sensado Kelvin en el borde interior (rev D)"
 			(at 116.84 40.64 0)
 			(hide yes)
@@
 			)
 		)
-		(property "Funcion" "Shunt de 1 mOhm (4 terminales) para medir la corriente total"
+		(property "Funcion" "Shunt de 1 mOhm 2 W (HoJLR2512, C2924520, en existencia) con sensado Kelvin en el borde interior (rev D)"
 			(at 116.84 40.64 0)
 			(hide yes)
@@
 			)
 		)
-		(property "Footprint" "RF_Module:ESP32-C3-WROOM-02"
+		(property "Footprint" "LetreroLab:ESP32-C3-WROOM-02_JLC"
 			(at 332.74 269.24 0)
 			(hide yes)
