File: hardware/ap1-base/kicad/AP1_Base.kicad_sch (KiCad schematic)
At the start: 65 parts, among them J1 ENTRADA 12-24V, J3 +V SALIDA, J4 CANALES, J5 FOCOS CC, J6 AUX 12V, J7 PROGRAMADOR, Q1 BSC028N06LS3, Q2 BSC028N06LS3, Q3 BSC028N06LS3, Q4 BSC028N06LS3, Q5 AO3400A, U1 INA238, U2 LMR16006XDDC, U3 UCC27524D, U4 UCC27524D, U6 AL8860MP, U7 AL8860MP, U8 TMP1075D, U9 AT24CS02

Commit message: AP-1 base a 4 capas, biblioteca JLCPCB y códigos LCSC automáticos
- placa.py: CAPAS=4 con planos internos (In1/In2 GND, tipo power para que
  Freerouting no rutee ahí), vías de costura GND (COSTURA) y zona sin cobre
  bajo la antena en todas las capas.
- AP1_Base: 4 capas JLC04161H-7628 (externas 2 oz, internas 1 oz), 61 vías de
  costura; ERC 0, DRC 0, 0 sin conectar, 0 diferencias.
- tools/jlcpcb.py + jlcpcb_catalogo.csv: 1499 piezas Basic/Preferred de la
  biblioteca JLCPCB-KiCad-Library (CDFER, MIT) y buscador por valor/huella.
- tools/descargar_biblioteca_jlcpcb.sh: instala la biblioteca para KiCad 9 y
  rehace el catálogo.
- salidas.py: BOM con LCSC y clase, RESUMEN_JLCPCB.txt con el cargo de piezas
  Extended, Gerber de todas las capas de cobre, PDF del lado inferior.
- Programador: D1/D2 SS14 -> B5819W (Preferred, misma huella).

Co-Authored-By: Claude Opus 5.5 <noreply@anthropic.com>
Claude-Session: https://claude.ai/code/session_01WVk3oGwfQfGTmAT2PMp8oW
Other:
- company: PCB 88 x 56 mm, 2 capas, cobre 2 oz recomendado -> PCB 88 x 56 mm, 4 capas JLC04161H-7628, externas 2 oz, internas 1 oz
Changed lines of the file:
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@@
 		(date "2026-10-01")
 		(rev "1.0")
-		(company "PCB 88 x 56 mm, 2 capas, cobre 2 oz recomendado")
-		(comment 1 "Placa de 2 capas para ensamble en fábrica (JLCPCB)")
+		(company "PCB 88 x 56 mm, 4 capas JLC04161H-7628, externas 2 oz, internas 1 oz")
+		(comment 1 "Placa de 4 capas (In1/In2 = GND) para ensamble en fábrica (JLCPCB)")
 		(comment 2 "12-24 V DC, 4 x 8 A + 2 x 1 A CC + AUX")
 	)

Commit message: AP-1: corte de MOSFET por hardware, supresor a la medida de los AL8860 y Home Assistant
- Base: la línea ALERTA (INA238 sobrecorriente/sobrevoltaje, TMP1075 85 C)
  apaga los dos UCC27524 por sus EN a través de D8/D9 (1N4148WS), sin
  depender del programa. Los diodos aíslan el pull-up interno de 12 V de los EN.
- Base: D1 SMBJ33A -> SMBJ26A. El anterior dejaba pasar hasta 53 V y los
  AL8860 aguantan 42 V; entrada máxima 26 V. Ruteada otra vez a 4 capas:
  ERC 0, DRC 0, 0 sin conectar, 0 diferencias.
- Programa fw 1.1: alerta del INA238 en menos de 1 ms (bus/temperatura a
  150 us), sobrevoltaje a 28 V, descubrimiento MQTT de Home Assistant (luz
  con brillo y efectos, AUX, focos CC, diagnóstico, sensores), varias órdenes
  por mensaje MQTT y 'O - b' para el foco 2 solo.

Co-Authored-By: Claude Opus 5.5 <noreply@anthropic.com>
Claude-Session: https://claude.ai/code/session_01WVk3oGwfQfGTmAT2PMp8oW
Parts:
- added D8, D9: 1N4148WS, Diode_SMD:D_SOD-323, symbol Device:D
- D1: value SMBJ33A -> SMBJ26A; Funcion Supresor de picos -> Supresor de picos: conduce desde 28.9 V y limita a 42 V, lo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
Connections:
- net ALERT: now also D8.1 (K), D9.1 (K)
- net EN12: now reaches U3.1 (ENA)
- net EN12: now also U3.8 (ENB), D8.2 (A)
- net EN34: now reaches U4.1 (ENA)
- net EN34: now also U4.8 (ENB), D9.2 (A)
- no-connect marks 6 -> 2
Other:
- moved on the sheet: C14, C15, C8, C9, D4, J4, J6, J7, Q1, Q2, Q3, Q4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

Commit message: Pedido más económico en JLCPCB: menos piezas Extended y BOM solo SMD
- Base: memoria AT24CS02 -> M24C02 (Preferred). El programa crea el número
  de serie (128 bits al azar con la MAC del programador) si la memoria no trae.
- Programador y AP-0.2: botones TL3342 -> TS-1187A (Basic, misma huella).
  En la AP-0.2 se cambió la huella sin volver a rutear: DRC 0.
- Base: rutas fijas para SWC1/SWC2 y CC2 igual que CC1 (el canal 2 es
  copia del 1, 12.5 mm abajo). Ruteo estable: ERC 0, DRC 0, 0 sin conectar.
- salidas.py: BOM/CPL '_solo_SMD' para soldar a mano clemas y conectores,
  resumen con cargo por código LCSC distinto y costo de piezas Basic.
- jlcpcb.py: piezas reconocidas por huella (botones con valor de etiqueta).
- Cargo de montaje por pedido: base+programador de ~93 a ~84 USD, o ~54 USD
  en el pedido solo SMD.

Co-Authored-By: Claude Opus 5.5 <noreply@anthropic.com>
Claude-Session: https://claude.ai/code/session_01WVk3oGwfQfGTmAT2PMp8oW
Parts:
- U9: value AT24CS02 -> M24C02-WMN6TP; footprint Package_TO_SOT_SMD:SOT-23-5 -> Package_SO:SOIC-8_3.9x4.9mm_P1.27mm; symbol Memory_EEPROM:AT24CS02-STUM -> Memory_EEPROM:M24C02-WMN; Funcion Identidad de la base: modelo, calibración y número de serie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 -> Identidad de la base: modelo, calibración, serie y horas (I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
Connections:
- net 3V3: now also U9.8 (VCC); no longer U9.4 (VCC)
- net GND: now also U9.1 (E0), U9.3 (E2), U9.4 (VSS), U9.7 (~{WC}); no longer U9.5 (WP)
- net SCL: now also U9.6 (SCL); no longer U9.1 (SCL)
- net SDA: now also U9.5 (SDA); no longer U9.3 (SDA)
Other:
- note added: "LetreroLab AP-1 BASE universal: 12-24 V / 20 A, 4 canales de 8 A, 2 canales de corriente constante (1 A), AUX 12 V. I2C: INA238 0x40, TMP1075 0x48, M24C02 0x50. 3V3 lo da el programador por J7."
- note removed: "LetreroLab AP-1 BASE universal: 12-24 V / 20 A, 4 canales de 8 A, 2 canales de corriente constante (1 A), AUX 12 V. I2C: INA238 0x40, TMP1075 0x48, AT24CS02 0x50 (+0x58 serie). 3V3 lo da el programador por J7."
Changed lines of the file:
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@@
 	(title_block
 		(title "LetreroLab AP-1 - base universal de potencia")
-		(date "2026-10-01")
+		(date "2026-10-02")
 		(rev "1.0")
 		(company "PCB 88 x 56 mm, 4 capas JLC04161H-7628, externas 2 oz, internas 1 oz")
@@
 	)
 	(symbol
-		(lib_id "Memory_EEPROM:AT24CS02-STUM")
+		(lib_id "Memory_EEPROM:M24C02-WMN")
 		(at 375.92 269.24 0)
 		(unit 1)
@@
 			)
 		)
-		(property "Value" "AT24CS02"
+		(property "Value" "M24C02-WMN6TP"
 			(at 398.08 270.84 0)
 			(effects
@@
 			)
 		)
-		(property "Footprint" "Package_TO_SOT_SMD:SOT-23-5"
+		(property "Footprint" "Package_SO:SOIC-8_3.9x4.9mm_P1.27mm"
 			(at 375.92 269.24 0)
 			(hide yes)
@@
 			)
 		)
-		(property "Description" "Identidad de la base: modelo, calibración y número de serie único (I2C 0x50/0x58)"
+		(property "Description" "Identidad de la base: modelo, calibración, serie y horas (I2C 0x50). Preferred de JLCPCB: sin cargo por tipo"
 			(at 375.92 269.24 0)
 			(hide yes)
@@
 			)
 		)
-		(property "Funcion" "Identidad de la base: modelo, calibración y número de serie único (I2C 0x50/0x58)"
+		(property "Funcion" "Identidad de la base: modelo, calibración, serie y horas (I2C 0x50). Preferred de JLCPCB: sin cargo por tipo"
 			(at 375.92 269.24 0)
 			(hide yes)
@@
 			)
 		)
-		(pin "4"
+		(pin "1"
 		)
 		(pin "2"
@@
 		(pin "3"
 		)
-		(pin "1"
+		(pin "8"
+		)
+		(pin "4"
 		)
 		(pin "5"
 		)
+		(pin "6"
+		)
+		(pin "7"
+		)
 		(instances
 			(project "AP1_Base"
@@
 	(wire
 		(pts
+			(xy 365.76 266.7)
+			(xy 363.22 266.7)
+		)
+		(stroke
+			(width 0)
+			(type default)
+		)
+	)
+	(label "GND"
+		(at 363.22 266.7 180)
+		(fields_autoplaced yes)
+		(effects
+			(font
+				(size 1.27 1.27)
+			)
+			(justify right bottom)
+		)
+	)
+	(wire
+		(pts
+			(xy 365.76 269.24)
+			(xy 363.22 269.24)
+		)
+		(stroke
+			(width 0)
+			(type default)
+		)
+	)
+	(label "GND"
+		(at 363.22 269.24 180)
+		(fields_autoplaced yes)
+		(effects
+			(font
+				(size 1.27 1.27)
+			)
+			(justify right bottom)
+		)
+	)
+	(wire
+		(pts
+			(xy 365.76 271.78)
+			(xy 363.22 271.78)
+		)
+		(stroke
+			(width 0)
+			(type default)
+		)
+	)
+	(label "GND"
+		(at 363.22 271.78 180)
+		(fields_autoplaced yes)
+		(effects
+			(font
+				(size 1.27 1.27)
+			)
+			(justify right bottom)
+		)
+	)
+	(wire
+		(pts
 			(xy 375.92 261.62)
 			(xy 375.92 259.08)
@@
 		)
 	)
-	(text "LetreroLab AP-1 BASE universal: 12-24 V / 20 A, 4 canales de 8 A, 2 canales de corriente constante (1 A), AUX 12 V.\nI2C: INA238 0x40, TMP1075 0x48, AT24CS02 0x50 (+0x58 serie). 3V3 lo da el programador por J7."
+	(text "LetreroLab AP-1 BASE universal: 12-24 V / 20 A, 4 canales de 8 A, 2 canales de corriente constante (1 A), AUX 12 V.\nI2C: INA238 0x40, TMP1075 0x48, M24C02 0x50. 3V3 lo da el programador por J7."
 		(exclude_from_sim no)
 		(at 150 15 0)

Commit message: Listo para JLCPCB: códigos LCSC, reglas de fabricación y carpeta de pedido
- Códigos LCSC verificados para todas las piezas SMD (INA238, LMR16006,
  UCC27524, AL8860, TMP1075, MOSFET, bobinas, capacitor, fusible, módulo,
  conectores) en tools/jlcpcb.py; piezas reconocidas por huella.
- Shunt: el WSK2512 de 4 terminales se agotó en LCSC; base y AP-0.2 usan un
  HoJLR2512 1 mOhm 2 W (C2924520) con huella propia 'net tie' que conserva
  el sensado Kelvin (tools/huellas/LetreroLab.pretty).
- ESP32-C3-WROOM-02: huella propia con 4 vías de 0.3 mm en lugar de 12 de
  0.2 mm (proceso estándar de JLCPCB). Textos de serigrafía de 0.8 mm o más.
- IND: fusible de 3 A (el mismo de la base).
- AP-0.2 ruteada otra vez con el nuevo shunt.
- Las 4 placas: ERC 0, DRC 0, 0 sin conectar, 0 diferencias y 0 problemas
  con las reglas de fabricación de JLCPCB.
- PEDIDO_JLCPCB/ (+ .zip) con Gerber, BOM y CPL completos o solo SMD por
  placa, y PEDIDO_JLCPCB.md con las opciones exactas del pedido.

Co-Authored-By: Claude Opus 5.5 <noreply@anthropic.com>
Claude-Session: https://claude.ai/code/session_01WVk3oGwfQfGTmAT2PMp8oW
Parts:
- RS1: value 1mR 2512 Kelvin -> 1mR 2512 2W; footprint Resistor_SMD:R_Shunt_Vishay_WSK2512_6332Metric_T1.19mm -> LetreroLab:R_2512_Kelvin_NetTie; Funcion Shunt de 1 mOhm con sensado Kelvin -> Shunt de 1 mOhm 2 W (HoJLR2512, C2924520, en existencia) co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
Changed lines of the file:
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@@
 			)
 		)
-		(property "Value" "1mR 2512 Kelvin"
+		(property "Value" "1mR 2512 2W"
 			(at 131.38 42.24 0)
 			(effects
@@
 			)
 		)
-		(property "Footprint" "Resistor_SMD:R_Shunt_Vishay_WSK2512_6332Metric_T1.19mm"
+		(property "Footprint" "LetreroLab:R_2512_Kelvin_NetTie"
 			(at 116.84 40.64 0)
 			(hide yes)
@@
 			)
 		)
-		(property "Description" "Shunt de 1 mOhm con sensado Kelvin"
+		(property "Description" "Shunt de 1 mOhm 2 W (HoJLR2512, C2924520, en existencia) con sensado Kelvin en el borde interior de cada terminal"
 			(at 116.84 40.64 0)
 			(hide yes)
@@
 			)
 		)
-		(property "Funcion" "Shunt de 1 mOhm con sensado Kelvin"
+		(property "Funcion" "Shunt de 1 mOhm 2 W (HoJLR2512, C2924520, en existencia) con sensado Kelvin en el borde interior de cada terminal"
 			(at 116.84 40.64 0)
 			(hide yes)

Commit message: AP CONNECT: sin borneras en todas las placas, placa nueva AP PRO AI4 y guía de fabricantes
- Borneras de tornillo reemplazadas por conectores con cable y código LCSC verificado:
  XT60 (C98732), JST VH 2/3/4 (C160315/6/7), JST XH 2/3/4 (C158012, C144394/5), Qwiic
  en BASE, IND, PIX, DMX, PLANTILLA, AP INPUT, AP OUTPUT y DIST 4; zonas de potencia rehechas
- XT60 de la DIST 4 con la polaridad marcada en la huella (pata 1 = -, pata 2 = +)
- TCA9554PWR ya con código (C477924)
- ap1-ai4: 4 entradas 0-10 V / 4-20 mA con ADS1115 (C37593), +24 V para sensores de lazo
- Programa 1.7: lectura AI4, umbrales con acciones, Home Assistant, tarjeta en la app
- FABRICANTES.md: JLCPCB, PCBWay, Seeed, NextPCB, México; impresión 3D y tornillería
- Pedido JLCPCB con 10 placas (AP-0.2 retirada); ERC/DRC/DFM 0 en todas

Co-Authored-By: Claude Opus 5.5 <noreply@anthropic.com>
Claude-Session: https://claude.ai/code/session_01WVk3oGwfQfGTmAT2PMp8oW
Parts:
- added J8: FOCO CC 2, Connector_JST:JST_XH_B2B-XH-A_1x02_P2.50mm_Vertical, symbol Connector_Generic:Conn_01x02
- J1: footprint TerminalBlock_Phoenix:TerminalBlock_Phoenix_MKDS-3-2-5.08_1x02_P5.08mm_Horizontal -> Connector_JST:JST_VH_B4P-VH_1x04_P3.96mm_Vertical; symbol Connector:Screw_Terminal_01x02 -> Connector_Generic:Conn_01x04; Funcion Entrada 12-24 V DC (+ / -), hasta 20 A -> Entrada 12-24 V DC: patas 1-2 = +, 3-4 = -, hasta 20 A (JST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
- J3: footprint TerminalBlock_Phoenix:TerminalBlock_Phoenix_MKDS-3-2-5.08_1x02_P5.08mm_Horizontal -> Connector_JST:JST_VH_B2P-VH_1x02_P3.96mm_Vertical; symbol Connector:Screw_Terminal_01x02 -> Connector_Generic:Conn_01x02; Funcion +12/24 V común de tiras y letreros (2 polos) -> +12/24 V común de tiras y letreros (2 patas, 20 A; JST VH)
- J4: footprint TerminalBlock_Phoenix:TerminalBlock_Phoenix_MKDS-3-4-5.08_1x04_P5.08mm_Horizontal -> Connector_JST:JST_VH_B4P-VH_1x04_P3.96mm_Vertical; symbol Connector:Screw_Terminal_01x04 -> Connector_Generic:Conn_01x04; Funcion Negativo conmutado de cada canal (8 A c/u) -> Negativo conmutado de cada canal (8 A c/u; JST VH, 10 A por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
- J5: value FOCOS CC -> FOCO CC 1; footprint TerminalBlock_Phoenix:TerminalBlock_Phoenix_PT-1,5-4-3.5-H_1x04_P3.50mm_Horizontal -> Connector_JST:JST_XH_B2B-XH-A_1x02_P2.50mm_Vertical; symbol Connector:Screw_Terminal_01x04 -> Connector_Generic:Conn_01x02; Funcion Salidas de corriente constante: + y - de cada foco (flotant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 -> Foco de corriente constante 1: 1 = +, 2 = - (flotante: no u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
- J6: footprint TerminalBlock_Phoenix:TerminalBlock_Phoenix_PT-1,5-2-3.5-H_1x02_P3.50mm_Horizontal -> Connector_JST:JST_XH_B2B-XH-A_1x02_P2.50mm_Vertical; symbol Connector:Screw_Terminal_01x02 -> Connector_Generic:Conn_01x02
Connections:
- net GNDIN: now also J1.3 (Pin_3), J1.4 (Pin_4); no longer J1.2 (Pin_2)
- net LEDA2: now also J8.1 (Pin_1); no longer J5.3 (Pin_3)
- net LEDK2: now also J8.2 (Pin_2); no longer J5.4 (Pin_4)
- net VIN_RAW: now also J1.2 (Pin_2)
Other:
- moved on the sheet: C11, C12, C14, C15, C8, C9, D2, D3, D4, D8, D9, J7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
