File: hardware/ap1-dist4/kicad/AP_Dist4.kicad_pcb (KiCad board)
At the start: 2 copper layers, 88 x 56 mm, 57 parts, among them J1 ENTRADA 12-24V, J2 RAMA 1, J3 RAMA 2, J4 RAMA 3, J5 RAMA 4, J6 QWIIC ENTRADA, J7 QWIIC SALIDA, U1 TCA9554PWR

Commit message: AP CONNECT: sin borneras en todas las placas, placa nueva AP PRO AI4 y guía de fabricantes
- Borneras de tornillo reemplazadas por conectores con cable y código LCSC verificado:
  XT60 (C98732), JST VH 2/3/4 (C160315/6/7), JST XH 2/3/4 (C158012, C144394/5), Qwiic
  en BASE, IND, PIX, DMX, PLANTILLA, AP INPUT, AP OUTPUT y DIST 4; zonas de potencia rehechas
- XT60 de la DIST 4 con la polaridad marcada en la huella (pata 1 = -, pata 2 = +)
- TCA9554PWR ya con código (C477924)
- ap1-ai4: 4 entradas 0-10 V / 4-20 mA con ADS1115 (C37593), +24 V para sensores de lazo
- Programa 1.7: lectura AI4, umbrales con acciones, Home Assistant, tarjeta en la app
- FABRICANTES.md: JLCPCB, PCBWay, Seeed, NextPCB, México; impresión 3D y tornillería
- Pedido JLCPCB con 10 placas (AP-0.2 retirada); ERC/DRC/DFM 0 en todas

Co-Authored-By: Claude Opus 5.5 <noreply@anthropic.com>
Claude-Session: https://claude.ai/code/session_01WVk3oGwfQfGTmAT2PMp8oW
Parts:
- J1: footprint TerminalBlock_Phoenix:TerminalBlock_Phoenix_MKDS-3-2-5.08_1x02_P5.08mm_Horizontal -> Connector_AMASS:AMASS_XT60PW-M_1x02_P7.20mm_Horizontal
- J2, J3, J4, J5: footprint TerminalBlock_Phoenix:TerminalBlock_Phoenix_MKDS-3-2-5.08_1x02_P5.08mm_Horizontal -> Connector_JST:JST_VH_B2P-VH_1x02_P3.96mm_Vertical
- moved J1 14.6 mm to (117.0, 144.0), turned to 90 degrees
- moved J2 3.55 mm to (123.5, 150.4)
- moved J3 3.55 mm to (139.5, 150.4)
- moved J4 3.55 mm to (155.5, 150.4)
- moved J5 3.55 mm to (171.5, 150.4)
- moved DG1 3.50 mm to (132.7, 134.6)
- moved DG2 3.50 mm to (148.7, 134.6)
- moved DG3 3.50 mm to (164.7, 134.6)
- moved DG4 3.50 mm to (180.7, 134.6)
- moved DR2 3.50 mm to (145.7, 134.6)
- moved DR3 3.50 mm to (161.7, 134.6)
- moved DR4 3.50 mm to (177.7, 134.6)
- moved F1 3.50 mm to (125.2, 124.0)
- moved F2 3.50 mm to (141.2, 124.0)
- moved F3 3.50 mm to (157.2, 124.0)
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Connections:
- J1 pad 1: /VIN -> /LGND
- J1 pad 2: /LGND -> /VIN
Routing:
- net /VIN: track 166.9 -> 136.3 mm, vias 1 -> 4
- net /GND: track 153.4 -> 134.3 mm, vias 27 -> 31
- net /SCL: track 47.7 -> 55.5 mm
- net /SEN1: track 20.4 -> 14.1 mm, vias 0 -> 2
- net /OUT2: track 45.4 -> 51.7 mm
- net /LGND: track 230.6 -> 236.3 mm, vias 74 -> 65
- net /SDA: track 49.8 -> 55.4 mm
- net /OUT4: track 44.5 -> 50.0 mm
- net /SENV: track 39.8 -> 34.8 mm, vias 0 -> 2
- net /SEN3: track 33.4 -> 37.5 mm, vias 2 -> 3
- net /OUT1: track 47.6 -> 51.6 mm, vias 2 -> 1
- net /OUT3: track 45.0 -> 48.3 mm
- net /SEN4: track 49.1 -> 52.3 mm
- net /SEN2: track 18.5 -> 20.8 mm, vias 2 -> 0
- net /A1: track 43.1 -> 41.3 mm
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Other:
- board text added: "ENTRADA 12-24V"
- board text added: "XT60"
- board text removed: "+"
