File: hardware/ap1-dist4/kicad/AP_Dist4.kicad_sch (KiCad schematic)
At the start: 54 parts, among them J1 ENTRADA 12-24V, J2 RAMA 1, J3 RAMA 2, J4 RAMA 3, J5 RAMA 4, J6 QWIIC ENTRADA, J7 QWIIC SALIDA, U1 TCA9554PWR

Commit message: AP CONNECT: sin borneras en todas las placas, placa nueva AP PRO AI4 y guía de fabricantes
- Borneras de tornillo reemplazadas por conectores con cable y código LCSC verificado:
  XT60 (C98732), JST VH 2/3/4 (C160315/6/7), JST XH 2/3/4 (C158012, C144394/5), Qwiic
  en BASE, IND, PIX, DMX, PLANTILLA, AP INPUT, AP OUTPUT y DIST 4; zonas de potencia rehechas
- XT60 de la DIST 4 con la polaridad marcada en la huella (pata 1 = -, pata 2 = +)
- TCA9554PWR ya con código (C477924)
- ap1-ai4: 4 entradas 0-10 V / 4-20 mA con ADS1115 (C37593), +24 V para sensores de lazo
- Programa 1.7: lectura AI4, umbrales con acciones, Home Assistant, tarjeta en la app
- FABRICANTES.md: JLCPCB, PCBWay, Seeed, NextPCB, México; impresión 3D y tornillería
- Pedido JLCPCB con 10 placas (AP-0.2 retirada); ERC/DRC/DFM 0 en todas

Co-Authored-By: Claude Opus 5.5 <noreply@anthropic.com>
Claude-Session: https://claude.ai/code/session_01WVk3oGwfQfGTmAT2PMp8oW
Parts:
- J1: footprint TerminalBlock_Phoenix:TerminalBlock_Phoenix_MKDS-3-2-5.08_1x02_P5.08mm_Horizontal -> Connector_AMASS:AMASS_XT60PW-M_1x02_P7.20mm_Horizontal; symbol Connector:Screw_Terminal_01x02 -> Connector_Generic:Conn_01x02; Funcion Fuente de los LED: + y 0 V (hasta 10 A) -> Fuente de los LED: XT60, + y - como las marcas del conector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
- J2, J3, J4, J5: footprint TerminalBlock_Phoenix:TerminalBlock_Phoenix_MKDS-3-2-5.08_1x02_P5.08mm_Horizontal -> Connector_JST:JST_VH_B2P-VH_1x02_P3.96mm_Vertical; symbol Connector:Screw_Terminal_01x02 -> Connector_Generic:Conn_01x02
Connections:
- net LGND: now also J1.1 (Pin_1); no longer J1.2 (Pin_2)
- net VIN: now also J1.2 (Pin_2); no longer J1.1 (Pin_1)
Changed lines of the file:
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@@
 	(title_block
 		(title "AP ELECTRIC · AP SIGN DIST 4 - distribución DC protegida")
-		(date "2026-10-05")
+		(date "2026-10-06")
 		(rev "1.0")
 		(company "PCB 88 x 56 mm, 2 capas, 2 oz")
@@
 	)
 	(symbol
-		(lib_id "Connector:Screw_Terminal_01x02")
+		(lib_id "Connector_Generic:Conn_01x02")
 		(at 116.84 78.74 0)
 		(unit 1)
@@
 			)
 		)
-		(property "Footprint" "TerminalBlock_Phoenix:TerminalBlock_Phoenix_MKDS-3-2-5.08_1x02_P5.08mm_Horizontal"
+		(property "Footprint" "Connector_AMASS:AMASS_XT60PW-M_1x02_P7.20mm_Horizontal"
 			(at 116.84 78.74 0)
 			(hide yes)
@@
 			)
 		)
-		(property "Description" "Fuente de los LED: + y 0 V (hasta 10 A)"
+		(property "Description" "Fuente de los LED: XT60, + y - como las marcas del conector (hasta 10 A)"
 			(at 116.84 78.74 0)
 			(hide yes)
@@
 			)
 		)
-		(property "Funcion" "Fuente de los LED: + y 0 V (hasta 10 A)"
+		(property "Funcion" "Fuente de los LED: XT60, + y - como las marcas del conector (hasta 10 A)"
 			(at 116.84 78.74 0)
 			(hide yes)
@@
 		)
 	)
-	(label "VIN"
+	(label "LGND"
 		(at 109.22 78.74 180)
 		(fields_autoplaced yes)
@@
 		)
 	)
-	(label "LGND"
+	(label "VIN"
 		(at 109.22 81.28 180)
 		(fields_autoplaced yes)
@@
 	)
 	(symbol
-		(lib_id "Connector:Screw_Terminal_01x02")
+		(lib_id "Connector_Generic:Conn_01x02")
 		(at 73.66 116.84 0)
 		(unit 1)
@@
 			)
 		)
-		(property "Footprint" "TerminalBlock_Phoenix:TerminalBlock_Phoenix_MKDS-3-2-5.08_1x02_P5.08mm_Horizontal"
+		(property "Footprint" "Connector_JST:JST_VH_B2P-VH_1x02_P3.96mm_Vertical"
 			(at 73.66 116.84 0)
 			(hide yes)
@@
 	)
 	(symbol
-		(lib_id "Connector:Screw_Terminal_01x02")
+		(lib_id "Connector_Generic:Conn_01x02")
 		(at 203.2 154.94 0)
 		(unit 1)
@@
 			)
 		)
-		(property "Footprint" "TerminalBlock_Phoenix:TerminalBlock_Phoenix_MKDS-3-2-5.08_1x02_P5.08mm_Horizontal"
+		(property "Footprint" "Connector_JST:JST_VH_B2P-VH_1x02_P3.96mm_Vertical"
 			(at 203.2 154.94 0)
 			(hide yes)
@@
 	)
 	(symbol
-		(lib_id "Connector:Screw_Terminal_01x02")
+		(lib_id "Connector_Generic:Conn_01x02")
 		(at 30.48 231.14 0)
 		(unit 1)
@@
 			)
 		)
-		(property "Footprint" "TerminalBlock_Phoenix:TerminalBlock_Phoenix_MKDS-3-2-5.08_1x02_P5.08mm_Horizontal"
+		(property "Footprint" "Connector_JST:JST_VH_B2P-VH_1x02_P3.96mm_Vertical"
 			(at 30.48 231.14 0)
 			(hide yes)
@@
 	)
 	(symbol
-		(lib_id "Connector:Screw_Terminal_01x02")
+		(lib_id "Connector_Generic:Conn_01x02")
 		(at 160.02 269.24 0)
 		(unit 1)
@@
 			)
 		)
-		(property "Footprint" "TerminalBlock_Phoenix:TerminalBlock_Phoenix_MKDS-3-2-5.08_1x02_P5.08mm_Horizontal"
+		(property "Footprint" "Connector_JST:JST_VH_B2P-VH_1x02_P3.96mm_Vertical"
 			(at 160.02 269.24 0)
 			(hide yes)
