File: hardware/ap1-dmx/kicad/AP1_DMX.kicad_sch (KiCad schematic)
At the start: 30 parts, among them J1 ENTRADA 12-24V, J2 DMX, J7 PROGRAMADOR, U1 M24C02-WMN6TP, U2 LMR16006XDDC, U3 SP3485EN

Commit message: AP CONNECT: sin borneras en todas las placas, placa nueva AP PRO AI4 y guía de fabricantes
- Borneras de tornillo reemplazadas por conectores con cable y código LCSC verificado:
  XT60 (C98732), JST VH 2/3/4 (C160315/6/7), JST XH 2/3/4 (C158012, C144394/5), Qwiic
  en BASE, IND, PIX, DMX, PLANTILLA, AP INPUT, AP OUTPUT y DIST 4; zonas de potencia rehechas
- XT60 de la DIST 4 con la polaridad marcada en la huella (pata 1 = -, pata 2 = +)
- TCA9554PWR ya con código (C477924)
- ap1-ai4: 4 entradas 0-10 V / 4-20 mA con ADS1115 (C37593), +24 V para sensores de lazo
- Programa 1.7: lectura AI4, umbrales con acciones, Home Assistant, tarjeta en la app
- FABRICANTES.md: JLCPCB, PCBWay, Seeed, NextPCB, México; impresión 3D y tornillería
- Pedido JLCPCB con 10 placas (AP-0.2 retirada); ERC/DRC/DFM 0 en todas

Co-Authored-By: Claude Opus 5.5 <noreply@anthropic.com>
Claude-Session: https://claude.ai/code/session_01WVk3oGwfQfGTmAT2PMp8oW
Parts:
- J1: footprint TerminalBlock_Phoenix:TerminalBlock_Phoenix_MKDS-3-2-5.08_1x02_P5.08mm_Horizontal -> Connector_JST:JST_VH_B2P-VH_1x02_P3.96mm_Vertical; symbol Connector:Screw_Terminal_01x02 -> Connector_Generic:Conn_01x02
- J2: footprint TerminalBlock_Phoenix:TerminalBlock_Phoenix_MKDS-3-3-5.08_1x03_P5.08mm_Horizontal -> Connector_JST:JST_XH_B3B-XH-A_1x03_P2.50mm_Vertical; symbol Connector:Screw_Terminal_01x03 -> Connector_Generic:Conn_01x03
Changed lines of the file:
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@@
 	(title_block
 		(title "LetreroLab AP-1 DMX512 - módulo para equipos DMX")
-		(date "2026-10-05")
+		(date "2026-10-06")
 		(rev "1.0")
 		(company "PCB 88 x 56 mm, 2 capas, 1 oz")
@@
 	)
 	(symbol
-		(lib_id "Connector:Screw_Terminal_01x02")
+		(lib_id "Connector_Generic:Conn_01x02")
 		(at 30.48 40.64 0)
 		(unit 1)
@@
 			)
 		)
-		(property "Footprint" "TerminalBlock_Phoenix:TerminalBlock_Phoenix_MKDS-3-2-5.08_1x02_P5.08mm_Horizontal"
+		(property "Footprint" "Connector_JST:JST_VH_B2P-VH_1x02_P3.96mm_Vertical"
 			(at 30.48 40.64 0)
 			(hide yes)
@@
 	)
 	(symbol
-		(lib_id "Connector:Screw_Terminal_01x03")
+		(lib_id "Connector_Generic:Conn_01x03")
 		(at 289.56 154.94 0)
 		(unit 1)
@@
 			)
 		)
-		(property "Footprint" "TerminalBlock_Phoenix:TerminalBlock_Phoenix_MKDS-3-3-5.08_1x03_P5.08mm_Horizontal"
+		(property "Footprint" "Connector_JST:JST_XH_B3B-XH-A_1x03_P2.50mm_Vertical"
 			(at 289.56 154.94 0)
 			(hide yes)
