File: hardware/ap1-ind/kicad/AP1_Industrial.kicad_sch (KiCad schematic)
At the start: 68 parts, among them J1 ENTRADA 12-24V, J2 CONTACTORES, J3 0-10V, J7 PROGRAMADOR, Q1 AO3400A, Q2 AO3400A, U1 LMR16006XDDC, U2 B1212S-1WR3, U3 LM358DR2G, U4 LM358DR2G, U5 M24C02-WMN6TP

Commit message: Listo para JLCPCB: códigos LCSC, reglas de fabricación y carpeta de pedido
- Códigos LCSC verificados para todas las piezas SMD (INA238, LMR16006,
  UCC27524, AL8860, TMP1075, MOSFET, bobinas, capacitor, fusible, módulo,
  conectores) en tools/jlcpcb.py; piezas reconocidas por huella.
- Shunt: el WSK2512 de 4 terminales se agotó en LCSC; base y AP-0.2 usan un
  HoJLR2512 1 mOhm 2 W (C2924520) con huella propia 'net tie' que conserva
  el sensado Kelvin (tools/huellas/LetreroLab.pretty).
- ESP32-C3-WROOM-02: huella propia con 4 vías de 0.3 mm en lugar de 12 de
  0.2 mm (proceso estándar de JLCPCB). Textos de serigrafía de 0.8 mm o más.
- IND: fusible de 3 A (el mismo de la base).
- AP-0.2 ruteada otra vez con el nuevo shunt.
- Las 4 placas: ERC 0, DRC 0, 0 sin conectar, 0 diferencias y 0 problemas
  con las reglas de fabricación de JLCPCB.
- PEDIDO_JLCPCB/ (+ .zip) con Gerber, BOM y CPL completos o solo SMD por
  placa, y PEDIDO_JLCPCB.md con las opciones exactas del pedido.

Co-Authored-By: Claude Opus 5.5 <noreply@anthropic.com>
Claude-Session: https://claude.ai/code/session_01WVk3oGwfQfGTmAT2PMp8oW
Parts:
- F1: value 2A -> 3A
Changed lines of the file:
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@@
 			)
 		)
-		(property "Value" "2A"
+		(property "Value" "3A"
 			(at 76.86 42.24 0)
 			(effects

Commit message: AP CONNECT: sin borneras en todas las placas, placa nueva AP PRO AI4 y guía de fabricantes
- Borneras de tornillo reemplazadas por conectores con cable y código LCSC verificado:
  XT60 (C98732), JST VH 2/3/4 (C160315/6/7), JST XH 2/3/4 (C158012, C144394/5), Qwiic
  en BASE, IND, PIX, DMX, PLANTILLA, AP INPUT, AP OUTPUT y DIST 4; zonas de potencia rehechas
- XT60 de la DIST 4 con la polaridad marcada en la huella (pata 1 = -, pata 2 = +)
- TCA9554PWR ya con código (C477924)
- ap1-ai4: 4 entradas 0-10 V / 4-20 mA con ADS1115 (C37593), +24 V para sensores de lazo
- Programa 1.7: lectura AI4, umbrales con acciones, Home Assistant, tarjeta en la app
- FABRICANTES.md: JLCPCB, PCBWay, Seeed, NextPCB, México; impresión 3D y tornillería
- Pedido JLCPCB con 10 placas (AP-0.2 retirada); ERC/DRC/DFM 0 en todas

Co-Authored-By: Claude Opus 5.5 <noreply@anthropic.com>
Claude-Session: https://claude.ai/code/session_01WVk3oGwfQfGTmAT2PMp8oW
Parts:
- removed J3: 0-10V, TerminalBlock_Phoenix:TerminalBlock_Phoenix_PT-1,5-8-3.5-H_1x08_P3.50mm_Horizontal, symbol Connector:Screw_Terminal_01x08
- added J4: K2, Connector_JST:JST_XH_B2B-XH-A_1x02_P2.50mm_Vertical, symbol Connector_Generic:Conn_01x02
- added J5: 0-10V 1, Connector_JST:JST_XH_B2B-XH-A_1x02_P2.50mm_Vertical, symbol Connector_Generic:Conn_01x02
- added J6: 0-10V 2, Connector_JST:JST_XH_B2B-XH-A_1x02_P2.50mm_Vertical, symbol Connector_Generic:Conn_01x02
- added J8: 0-10V 3, Connector_JST:JST_XH_B2B-XH-A_1x02_P2.50mm_Vertical, symbol Connector_Generic:Conn_01x02
- added J9: 0-10V 4, Connector_JST:JST_XH_B2B-XH-A_1x02_P2.50mm_Vertical, symbol Connector_Generic:Conn_01x02
- F1: Funcion Fusible de la placa -> Fusible de la placa (el mismo de la base)
- J1: footprint TerminalBlock_Phoenix:TerminalBlock_Phoenix_MKDS-3-2-5.08_1x02_P5.08mm_Horizontal -> Connector_JST:JST_VH_B2P-VH_1x02_P3.96mm_Vertical; symbol Connector:Screw_Terminal_01x02 -> Connector_Generic:Conn_01x02; Funcion Entrada 12-24 V DC (+ / -), máx. 26 V -> Entrada 12-24 V DC: 1 = +, 2 = -, máx. 26 V (JST VH)
- J2: value CONTACTORES -> K1; footprint TerminalBlock_Phoenix:TerminalBlock_Phoenix_PT-1,5-4-3.5-H_1x04_P3.50mm_Horizontal -> Connector_JST:JST_XH_B2B-XH-A_1x02_P2.50mm_Vertical; symbol Connector:Screw_Terminal_01x04 -> Connector_Generic:Conn_01x02; Funcion Bobina del contactor 1 y 2 (+V y salida conmutada), 0.5 A c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 -> Bobina del contactor 1: 1 = +V, 2 = salida conmutada, 0.5 A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
Connections:
- net DIM1: now also J5.1 (Pin_1)
- net DIM2: now also J6.1 (Pin_1)
- net DIM3: now also J8.1 (Pin_1)
- net DIM4: now also J9.1 (Pin_1)
- net ISOGND: now also J5.2 (Pin_2), J6.2 (Pin_2), J8.2 (Pin_2), J9.2 (Pin_2)
- net K2: now also J4.2 (Pin_2); no longer J2.4 (Pin_4)
- net VIN: now also J4.1 (Pin_1); no longer J2.3 (Pin_3)
Other:
- moved on the sheet: C10, C6, C7, C8, C9, CF1, CF2, CF3, CF4, D4, D5, DZ1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
