File: hardware/ap1-out/kicad/AP_Output.kicad_pcb (KiCad board)
At the start: 2 copper layers, 72 x 56 mm, 39 parts, among them J1 QWIIC ENTRADA, J2 QWIIC SALIDA, J3 I2C, J4 24V, J5 Q1-Q3, J6 Q4-Q6, J7 Q7 +24 +24, U1 TCA9554PWR, U2 ULN2003ADR

Commit message: AP CONNECT: sin borneras en todas las placas, placa nueva AP PRO AI4 y guía de fabricantes
- Borneras de tornillo reemplazadas por conectores con cable y código LCSC verificado:
  XT60 (C98732), JST VH 2/3/4 (C160315/6/7), JST XH 2/3/4 (C158012, C144394/5), Qwiic
  en BASE, IND, PIX, DMX, PLANTILLA, AP INPUT, AP OUTPUT y DIST 4; zonas de potencia rehechas
- XT60 de la DIST 4 con la polaridad marcada en la huella (pata 1 = -, pata 2 = +)
- TCA9554PWR ya con código (C477924)
- ap1-ai4: 4 entradas 0-10 V / 4-20 mA con ADS1115 (C37593), +24 V para sensores de lazo
- Programa 1.7: lectura AI4, umbrales con acciones, Home Assistant, tarjeta en la app
- FABRICANTES.md: JLCPCB, PCBWay, Seeed, NextPCB, México; impresión 3D y tornillería
- Pedido JLCPCB con 10 placas (AP-0.2 retirada); ERC/DRC/DFM 0 en todas

Co-Authored-By: Claude Opus 5.5 <noreply@anthropic.com>
Claude-Session: https://claude.ai/code/session_01WVk3oGwfQfGTmAT2PMp8oW
Parts:
- added J10: Q6, Connector_JST:JST_XH_B2B-XH-A_1x02_P2.50mm_Vertical, F.Cu at (155.5, 151.0)
- added J11: Q7, Connector_JST:JST_XH_B2B-XH-A_1x02_P2.50mm_Vertical, F.Cu at (164.1, 151.0)
- added J8: Q4, Connector_JST:JST_XH_B2B-XH-A_1x02_P2.50mm_Vertical, F.Cu at (138.3, 151.0)
- added J9: Q5, Connector_JST:JST_XH_B2B-XH-A_1x02_P2.50mm_Vertical, F.Cu at (146.9, 151.0)
- J4: footprint TerminalBlock_Phoenix:TerminalBlock_Phoenix_MKDS-3-2-5.08_1x02_P5.08mm_Horizontal -> Connector_JST:JST_VH_B2P-VH_1x02_P3.96mm_Vertical
- J5: value Q1-Q3 -> Q1; footprint TerminalBlock_Phoenix:TerminalBlock_Phoenix_MKDS-3-3-5.08_1x03_P5.08mm_Horizontal -> Connector_JST:JST_XH_B2B-XH-A_1x02_P2.50mm_Vertical
- J6: value Q4-Q6 -> Q2; footprint TerminalBlock_Phoenix:TerminalBlock_Phoenix_MKDS-3-3-5.08_1x03_P5.08mm_Horizontal -> Connector_JST:JST_XH_B2B-XH-A_1x02_P2.50mm_Vertical
- J7: value Q7 +24 +24 -> Q3; footprint TerminalBlock_Phoenix:TerminalBlock_Phoenix_MKDS-3-3-5.08_1x03_P5.08mm_Horizontal -> Connector_JST:JST_XH_B2B-XH-A_1x02_P2.50mm_Vertical
- moved J7 20.3 mm to (129.7, 151.0)
- moved DL6 13.6 mm to (156.8, 139.6)
- moved RL6 13.6 mm to (156.8, 135.6)
- moved DL7 13.1 mm to (163.1, 139.6)
- moved RL7 13.1 mm to (163.1, 135.6)
- moved J6 12.0 mm to (121.1, 151.0)
- moved DL5 10.1 mm to (148.2, 139.6)
- moved RL5 10.1 mm to (148.2, 135.6)
- moved DL4 6.55 mm to (139.6, 139.6)
- moved RL4 6.55 mm to (139.6, 135.6)
- moved DL3 4.79 mm to (130.9, 139.6)
- moved RL3 4.79 mm to (130.9, 135.6)
- moved J5 3.70 mm to (112.5, 151.0)
- moved DL1 2.25 mm to (113.8, 139.6)
- moved RL1 2.25 mm to (113.8, 135.6)
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Connections:
- J5 pad 1: /Q1 -> /V24
- J5 pad 2: /Q2 -> /Q1
- J6 pad 1: /Q4 -> /V24
- J6 pad 2: /Q5 -> /Q2
- J7 pad 1: /Q7 -> /V24
- J7 pad 2: /V24 -> /Q3
Routing:
- net /V24: track 134.4 -> 194.5 mm, vias 5 -> 4
- net /IN5: track 33.6 -> 13.6 mm, vias 4 -> 0
- net /Q7: track 30.7 -> 43.9 mm
- net /Q6: track 32.7 -> 45.1 mm
- net /SCL: track 58.0 -> 68.4 mm, vias 0 -> 1
- net /IN2: track 20.8 -> 29.4 mm, vias 0 -> 2
- net /3V3: track 92.1 -> 99.3 mm
- net /IN4: track 25.9 -> 19.2 mm
- net /Q5: track 33.7 -> 39.3 mm
- net /SDA: track 63.4 -> 67.3 mm
- net /Q1: track 48.9 -> 52.5 mm
- net /A0: track 20.4 -> 17.0 mm, vias 2 -> 0
- net /LA1: track 4.73 -> 7.59 mm, vias 0 -> 2
- net /IN1: track 21.2 -> 18.9 mm, vias 0 -> 2
- net /IN6: track 15.3 -> 16.9 mm
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Other:
- board text added: "+24 0V"
- board text added: "Carga entre las 2 patas de Qn. Red: solo con contactor"
- board text removed: "+24"
- board text removed: "0V"
- board text removed: "Carga entre +24 y Qn. Red: solo con contactor"
