File: hardware/ap1-plantilla/kicad/AP1_Plantilla.kicad_pcb (KiCad board)
At the start: 2 copper layers, 88 x 56 mm, 26 parts, among them J1 ENTRADA 12-24V, J7 PROGRAMADOR, J8 SEÑALES LL, U1 M24C02-WMN6TP, U2 LMR16006XDDC

Commit message: AP CONNECT: sin borneras en todas las placas, placa nueva AP PRO AI4 y guía de fabricantes
- Borneras de tornillo reemplazadas por conectores con cable y código LCSC verificado:
  XT60 (C98732), JST VH 2/3/4 (C160315/6/7), JST XH 2/3/4 (C158012, C144394/5), Qwiic
  en BASE, IND, PIX, DMX, PLANTILLA, AP INPUT, AP OUTPUT y DIST 4; zonas de potencia rehechas
- XT60 de la DIST 4 con la polaridad marcada en la huella (pata 1 = -, pata 2 = +)
- TCA9554PWR ya con código (C477924)
- ap1-ai4: 4 entradas 0-10 V / 4-20 mA con ADS1115 (C37593), +24 V para sensores de lazo
- Programa 1.7: lectura AI4, umbrales con acciones, Home Assistant, tarjeta en la app
- FABRICANTES.md: JLCPCB, PCBWay, Seeed, NextPCB, México; impresión 3D y tornillería
- Pedido JLCPCB con 10 placas (AP-0.2 retirada); ERC/DRC/DFM 0 en todas

Co-Authored-By: Claude Opus 5.5 <noreply@anthropic.com>
Claude-Session: https://claude.ai/code/session_01WVk3oGwfQfGTmAT2PMp8oW
Parts:
- J1: footprint TerminalBlock_Phoenix:TerminalBlock_Phoenix_MKDS-3-2-5.08_1x02_P5.08mm_Horizontal -> Connector_JST:JST_VH_B2P-VH_1x02_P3.96mm_Vertical
- moved J1 0.85 mm to (103.0, 150.4)
Routing:
- net /PWM3: track 73.4 -> 44.4 mm
- net /PWM1: track 51.8 -> 67.4 mm
- net /GND: track 207.7 -> 220.2 mm, vias 77 -> 79
- net /SDA: track 65.3 -> 56.3 mm
- net /PWM4: track 41.9 -> 49.4 mm, vias 0 -> 1
- net /SCL: track 63.8 -> 57.3 mm
- net /V12: track 117.3 -> 111.3 mm, vias 1 -> 0
- net /VIN: track 86.1 -> 83.9 mm, vias 3 -> 4
- net /ALERT: track 47.3 -> 45.4 mm, vias 1 -> 0
- net /VIN_RAW: track 12.7 -> 13.6 mm
- net /CC2: track 44.3 -> 44.7 mm, vias 0 -> 1
Other:
- board text added: "1+ 2-"
- board text removed: "+"
- board text removed: "-"
