File: hardware/ap-electric/7r-tour/kicad/AP_7R_TOUR.kicad_sch (KiCad schematic)
At the start: 181 parts, among them J1 KF128-5.08-2P, J11 KF128-5.08-3P, J12 KF128-5.08-3P, J13 KF128-5.08-3P, J14 KF128-5.08-3P, J15 USB-C, J2 KF128-5.08-2P, J3 KF128-5.08-2P, J4 KF128-5.08-2P, J5 KF128-5.08-2P, J6 KF128-5.08-2P, J7 KF128-5.08-2P, J8 KF128-5.08-2P, J9 KF128-5.08-2P, K1 G2RL-1A-E DC24, K2 G2RL-1A-E DC24, K3 G2RL-1A-E DC24, K4 G2RL-1A-E DC24, K5 G2RL-1A-E DC24, K6 G2RL-1A-E DC24, K7 G2RL-1A-E DC24, SW1 DSWB08LHGET, SW8 MODO, SW9 RESET, U1 ULN2003ADR, U10 USBLC6-2SC6, U2 TCA9554PWR, U3 TCA9554PWR, U4 TCA9554PWR, U5 TCA9554PWR, U6 CA-IS3092W, U7 LMR16006XDDC, U8 AP63203WU, U9 ESP32-C3-WROOM-02

Commit message: 7R Tour rev B: placa ruteada y cerrada (conteo rapido, reloj, puntos de prueba), buscador de caminos para 3 redes largas, BOM/CPL regenerados
Co-Authored-By: Claude Sonnet 5.5 <noreply@anthropic.com>
Claude-Session: https://claude.ai/code/session_01WVk3oGwfQfGTmAT2PMp8oW
Parts:
- added C28: 100nF, Capacitor_SMD:C_0603_1608Metric, symbol Device:C
- added D12: BAT54C, Package_TO_SOT_SMD:SOT-23, symbol Diode:BAT54C
- added J16: BAT, Connector_PinHeader_2.54mm:PinHeader_1x02_P2.54mm_Vertical, symbol Connector_Generic:Conn_01x02
- added TP1: TP 24V, TestPoint:TestPoint_Pad_D1.5mm, symbol Connector:TestPoint
- added TP10: TP DE, TestPoint:TestPoint_Pad_D1.5mm, symbol Connector:TestPoint
- added TP11: TP EN, TestPoint:TestPoint_Pad_D1.5mm, symbol Connector:TestPoint
- added TP2: TP 5V, TestPoint:TestPoint_Pad_D1.5mm, symbol Connector:TestPoint
- added TP3: TP 3V3, TestPoint:TestPoint_Pad_D1.5mm, symbol Connector:TestPoint
- added TP4, TP5: TP GND, TestPoint:TestPoint_Pad_D1.5mm, symbol Connector:TestPoint
- added TP6: TP SDA, TestPoint:TestPoint_Pad_D1.5mm, symbol Connector:TestPoint
- added TP7: TP SCL, TestPoint:TestPoint_Pad_D1.5mm, symbol Connector:TestPoint
- added TP8: TP TX, TestPoint:TestPoint_Pad_D1.5mm, symbol Connector:TestPoint
- added TP9: TP RX, TestPoint:TestPoint_Pad_D1.5mm, symbol Connector:TestPoint
- added U11: PCF8563T/5,518, Package_SO:SOIC-8_3.9x4.9mm_P1.27mm, symbol Timer_RTC:PCF8563T
- added Y1: 32.768kHz 12.5pF, Crystal:Crystal_SMD_3215-2Pin_3.2x1.5mm, symbol Device:Crystal
- U9: Funcion Wi-Fi opcional; IO2/IO8 = I2C, IO1/IO3/IO10 = RS-485, IO4 = interrupción de entradas y botones -> Wi-Fi opcional; IO2/IO8 = I2C, IO1/IO3/IO10 = RS-485, IO4 = interrupción de entradas y botones; IO0 e IO20 = conteo rápido de las entradas 1 y 2
Connections:
- net 3V3: now also D12.1, TP3.1
- net E1: now also U9.18 (IO0)
- net E2: now also U9.11 (IO20/RXD)
- net EN: now also TP11.1
- net GND: now also C28.2, J16.2 (Pin_2), TP4.1, TP5.1, U11.4 (VSS)
- net RS_DE: now also TP10.1
- net RS_RX: now also TP9.1
- net RS_TX: now also TP8.1
- net SCL: now also TP7.1, U11.6 (SCL)
- net SDA: now also TP6.1, U11.5 (SDA)
- net V24: now also TP1.1
- net V5: now also TP2.1
- new net OSCI: U11.1 (OSCI), Y1.1
- new net OSCO: U11.2 (OSCO), Y1.2
- new net VBAT: D12.2, J16.1 (Pin_1)
- new net VRTC: C28.1, D12.3, U11.8 (VDD)
Other:
- note added: "AP Electric Industrial · 7R Tour rev B (CONCEPTO): 7 x G2RL-1A-E 24 V, ULN2003A, 4 x TCA9554 (0x20-0x23), 8 entradas 24 V LTV-217, CA-IS3092W RS-485 aislado, ESP32-C3. SKU CA: IRM-20-24 + T2A + 10D471K. Rev B: conteo rápido en IO0/IO20 (entradas 1 y 2), reloj PCF8563T con batería externa, 11 puntos de prueba."
- note removed: "AP Electric Industrial · 7R Tour rev A (CONCEPTO): 7 x G2RL-1A-E 24 V, ULN2003A, 4 x TCA9554 (0x20-0x23), 8 entradas 24 V LTV-217, CA-IS3092W RS-485 aislado, ESP32-C3. SKU CA: IRM-20-24 + T2A + 10D471K."
- title: AP Electric Industrial · 7R Tour rev A - 7 relés, 8 entradas, Modbus aislado (CONCEPTO) -> AP Electric Industrial · 7R Tour rev B - 7 relés, 8 entradas, Modbus aislado (CONCEPTO)
- moved on the sheet: C20, C21, C22, C23, C24, C25, C26, C27, D11, DI1, DI2, DI3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

Commit message: 7R Tour rev B cerrada con pull-downs RD1-RD7: ERC 0, DRC 0, sin conectar 0, DFM 0; poda de ramas sin salida en ruta_auto; BOM/CPL, renders y vistas regenerados
Co-Authored-By: Claude Sonnet 5.5 <noreply@anthropic.com>
Claude-Session: https://claude.ai/code/session_01WVk3oGwfQfGTmAT2PMp8oW
Parts:
- added RD1, RD2, RD3, RD4, RD5, RD6, RD7: 10k, Resistor_SMD:R_0603_1608Metric, symbol Device:R
Connections:
- net DO1: now also RD1.1
- net DO2: now also RD2.1
- net DO3: now also RD3.1
- net DO4: now also RD4.1
- net DO5: now also RD5.1
- net DO6: now also RD6.1
- net DO7: now also RD7.1
- net GND: now also RD1.2, RD2.2, RD3.2, RD4.2, RD5.2, RD6.2, RD7.2
Other:
- moved on the sheet: DI1, DI2, DI3, DI4, DI5, DI6, DI7, DI8, J2, J3, J4, J5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

Commit message: Segunda ronda de correcciones: ciclo nominal en PK ENT, fallas I2C separadas, FABRICA solo local y con maniobras conservadas, consola USB con lineas completas, clave con ruido de hardware, vigilancia como latido de escrituras; web sin falsas promesas, datos malformados, doble envio, estados unificados, 30 V, contraste; consola con indicador de datos viejos y confirmaciones; AP Studio con clave; C14 a 10uF 50V
Co-Authored-By: Claude Sonnet 5.5 <noreply@anthropic.com>
Claude-Session: https://claude.ai/code/session_01WVk3oGwfQfGTmAT2PMp8oW
Parts:
- C14: value 10uF 25V -> 10uF 50V
Changed lines of the file:
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@@
 	(title_block
 		(title "AP Electric Industrial · 7R Tour rev B - 7 relés, 8 entradas, Modbus aislado (CONCEPTO)")
-		(date "2026-10-14")
+		(date "2026-10-15")
 		(rev "1.0")
 		(company "PCB 176 x 90 mm, 2 capas, 2 oz")
@@
 			)
 		)
-		(property "Value" "10uF 25V"
+		(property "Value" "10uF 50V"
 			(at 206.4 118.44 0)
 			(effects
