File: hardware/ap-electric/rack16/kicad/AP_RACK16.kicad_pcb (KiCad board)
At the start: 2 copper layers, 176 x 100 mm, 247 parts, among them J1 VIN 12-30V, J10 KF128-5.08-3P, J11 KF128-5.08-3P, J12 KF128-5.08-3P, J13 KF128-5.08-3P, J2 USB-C, J3 KF128-5.08-3P, J4 KF128-5.08-3P, J5 KF128-5.08-3P, J6 KF128-5.08-3P, J7 KF128-5.08-3P, J8 KF128-5.08-3P, J9 KF128-5.08-3P, Q1 NCV8406ASTT3G, Q10 NCV8406ASTT3G, Q11 NCV8406ASTT3G, Q12 NCV8406ASTT3G, Q13 NCV8406ASTT3G, Q14 NCV8406ASTT3G, Q15 NCV8406ASTT3G, Q16 NCV8406ASTT3G, Q2 NCV8406ASTT3G, Q3 NCV8406ASTT3G, Q4 NCV8406ASTT3G, Q5 NCV8406ASTT3G, Q6 NCV8406ASTT3G, Q7 NCV8406ASTT3G, Q8 NCV8406ASTT3G, Q9 NCV8406ASTT3G, SW1 MODO, SW2 RESET, U1 LMR16006XDDC, U10 74HCT125D, U11 74HCT125D, U12 74HCT125D, U13 74HCT125D, U2 AP63203WU, U3 ESP32-C3-WROOM-02, U4 USBLC6-2SC6, U5 SP3485EN, U6 TCA9554PWR, U7 TCA9554PWR, U8 TCA9554PWR, U9 TCA9554PWR

Commit message: AP Rack 16 rev A: placa cerrada (ERC/DRC/DFM 0), vistas, documentos y entrada de catálogo
Co-Authored-By: Claude Sonnet 5.5 <noreply@anthropic.com>
Claude-Session: https://claude.ai/code/session_01WVk3oGwfQfGTmAT2PMp8oW
Parts:
- F1: value MINI 10A -> MINI 3A
Routing:
- net /GND: track 0.00 -> 970.6 mm, vias 0 -> 376
- net /V24: track 0.00 -> 557.1 mm, vias 0 -> 7
- net /3V3: track 0.00 -> 384.1 mm, vias 0 -> 18
- net /V5: track 0.00 -> 270.0 mm, vias 0 -> 11
- net /SDA: track 0.00 -> 215.9 mm, vias 0 -> 8
- net /SCL: track 0.00 -> 180.9 mm, vias 0 -> 5
- net /RSA: track 0.00 -> 144.7 mm, vias 0 -> 2
- net /RSB: track 0.00 -> 143.1 mm, vias 0 -> 4
- net /SENSE_I: track 0.00 -> 134.3 mm, vias 0 -> 4
- net /COMI: track 0.00 -> 122.1 mm, vias 0 -> 8
- net /RS_DE: track 0.00 -> 110.8 mm
- net /INT: track 0.00 -> 110.0 mm, vias 0 -> 4
- net /RS_RX: track 0.00 -> 99.9 mm, vias 0 -> 2
- net /SENSE_O: track 0.00 -> 99.1 mm, vias 0 -> 3
- net /RS_TX: track 0.00 -> 94.0 mm, vias 0 -> 2
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- added copper zone on B.Cu, net /GND
- added copper zone on F.Cu, net /GND
Other:
- board text added: "+V 0V"
- board text added: "AP ELECTRIC AP RACK 16 rev A - CONCEPTO. 12-30 V CC. Carga entre +V y la salida. Red solo con contactor. SENSE/A/B: solo AP LINK, no AP BUS."
- board text added: "AP ELECTRIC INDUSTRIAL AP RACK 16 rev A"
- board text added: "ENTRA"
- board text added: "I1 I2 I3 I4 I5 I6 I7 I8 COM"
- board text added: "MODULO 8 4 2 1"
- board text added: "RUN FALLA COM CABEZA"
- board text added: "SIGUE"
