File: hardware/ap-electric/rack16/kicad/AP_RACK16.kicad_sch (KiCad schematic)
At the start: 243 parts, among them J1 VIN 12-30V, J10 KF128-5.08-3P, J11 KF128-5.08-3P, J12 KF128-5.08-3P, J13 KF128-5.08-3P, J2 USB-C, J3 KF128-5.08-3P, J4 KF128-5.08-3P, J5 KF128-5.08-3P, J6 KF128-5.08-3P, J7 KF128-5.08-3P, J8 KF128-5.08-3P, J9 KF128-5.08-3P, Q1 NCV8406ASTT3G, Q10 NCV8406ASTT3G, Q11 NCV8406ASTT3G, Q12 NCV8406ASTT3G, Q13 NCV8406ASTT3G, Q14 NCV8406ASTT3G, Q15 NCV8406ASTT3G, Q16 NCV8406ASTT3G, Q2 NCV8406ASTT3G, Q3 NCV8406ASTT3G, Q4 NCV8406ASTT3G, Q5 NCV8406ASTT3G, Q6 NCV8406ASTT3G, Q7 NCV8406ASTT3G, Q8 NCV8406ASTT3G, Q9 NCV8406ASTT3G, SW1 MODO, SW2 RESET, U1 LMR16006XDDC, U10 74HCT125D, U11 74HCT125D, U12 74HCT125D, U13 74HCT125D, U2 AP63203WU, U3 ESP32-C3-WROOM-02, U4 USBLC6-2SC6, U5 SP3485EN, U6 TCA9554PWR, U7 TCA9554PWR, U8 TCA9554PWR, U9 TCA9554PWR

Commit message: AP Rack 16 rev A: placa cerrada (ERC/DRC/DFM 0), vistas, documentos y entrada de catálogo
Co-Authored-By: Claude Sonnet 5.5 <noreply@anthropic.com>
Claude-Session: https://claude.ai/code/session_01WVk3oGwfQfGTmAT2PMp8oW
Parts:
- F1: value MINI 10A -> MINI 3A; Funcion Fusible mini de auto (ATM); se cambia sin soldar. Valor seg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 -> Fusible mini de auto (ATM) de 3 A en esta revisión: el +V d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
Changed lines of the file:
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@@
 			)
 		)
-		(property "Value" "MINI 10A"
+		(property "Value" "MINI 3A"
 			(at 76.86 42.24 0)
 			(effects
@@
 			)
 		)
-		(property "Description" "Fusible mini de auto (ATM); se cambia sin soldar. Valor según la carga total"
+		(property "Description" "Fusible mini de auto (ATM) de 3 A en esta revisión: el +V de la placa va en pistas de 0.8 mm (sin medir); se cambia sin soldar"
 			(at 73.66 40.64 0)
 			(hide yes)
@@
 			)
 		)
-		(property "Funcion" "Fusible mini de auto (ATM); se cambia sin soldar. Valor según la carga total"
+		(property "Funcion" "Fusible mini de auto (ATM) de 3 A en esta revisión: el +V de la placa va en pistas de 0.8 mm (sin medir); se cambia sin soldar"
 			(at 73.66 40.64 0)
 			(hide yes)
@@
 	(symbol
 		(lib_id "power:PWR_FLAG")
-		(at 20.32 20.32 0)
+		(at 96.52 20.32 0)
 		(unit 1)
 		(exclude_from_sim no)
@@
 		(dnp no)
 		(property "Reference" "#FLG01"
+			(at 99.72 19.32 0)
+			(hide yes)
+			(effects
+				(font
+					(size 1.27 1.27)
+				)
+				(justify left)
+			)
+		)
+		(property "Value" "PWR_FLAG"
+			(at 99.72 21.92 0)
+			(effects
+				(font
+					(size 1.27 1.27)
+				)
+				(justify left)
+			)
+		)
+		(property "Footprint" ""
+			(at 96.52 20.32 0)
+			(hide yes)
+			(effects
+				(font
+					(size 1.27 1.27)
+				)
+				(justify left)
+			)
+		)
+		(property "Datasheet" "~"
+			(at 96.52 20.32 0)
+			(hide yes)
+			(effects
+				(font
+					(size 1.27 1.27)
+				)
+				(justify left)
+			)
+		)
+		(property "Description" "Bandera de alimentación para ERC"
+			(at 96.52 20.32 0)
+			(hide yes)
+			(effects
+				(font
+					(size 1.27 1.27)
+				)
+				(justify left)
+			)
+		)
+		(pin "1"
+		)
+		(instances
+			(project "AP_RACK16"
+				(path "/8e2a4c6d-0f1b-4d3e-9a5c-7b9d1f3e5a64"
+					(reference "#FLG01")
+					(unit 1)
+				)
+			)
+		)
+	)
+	(wire
+		(pts
+			(xy 96.52 20.32)
+			(xy 96.52 22.86)
+		)
+		(stroke
+			(width 0)
+			(type default)
+		)
+	)
+	(label "GND"
+		(at 96.52 22.86 0)
+		(fields_autoplaced yes)
+		(effects
+			(font
+				(size 1.27 1.27)
+			)
+			(justify left bottom)
+		)
+	)
+	(symbol
+		(lib_id "power:PWR_FLAG")
+		(at 20.32 20.32 0)
+		(unit 1)
+		(exclude_from_sim no)
+		(in_bom no)
+		(on_board no)
+		(dnp no)
+		(property "Reference" "#FLG02"
 			(at 23.52 19.32 0)
 			(hide yes)
@@
 			(project "AP_RACK16"
 				(path "/8e2a4c6d-0f1b-4d3e-9a5c-7b9d1f3e5a64"
-					(reference "#FLG01")
+					(reference "#FLG02")
 					(unit 1)
 				)
@@
 		(on_board no)
 		(dnp no)
-		(property "Reference" "#FLG02"
+		(property "Reference" "#FLG03"
 			(at 38.76 19.32 0)
 			(hide yes)
@@
 			(project "AP_RACK16"
 				(path "/8e2a4c6d-0f1b-4d3e-9a5c-7b9d1f3e5a64"
-					(reference "#FLG02")
+					(reference "#FLG03")
 					(unit 1)
 				)
@@
 		(on_board no)
 		(dnp no)
-		(property "Reference" "#FLG03"
+		(property "Reference" "#FLG04"
 			(at 54 19.32 0)
 			(hide yes)
@@
 			(project "AP_RACK16"
 				(path "/8e2a4c6d-0f1b-4d3e-9a5c-7b9d1f3e5a64"
-					(reference "#FLG03")
+					(reference "#FLG04")
 					(unit 1)
 				)
@@
 		(on_board no)
 		(dnp no)
-		(property "Reference" "#FLG04"
+		(property "Reference" "#FLG05"
 			(at 69.24 19.32 0)
 			(hide yes)
@@
 			(project "AP_RACK16"
 				(path "/8e2a4c6d-0f1b-4d3e-9a5c-7b9d1f3e5a64"
-					(reference "#FLG04")
+					(reference "#FLG05")
 					(unit 1)
 				)
@@
 		(on_board no)
 		(dnp no)
-		(property "Reference" "#FLG05"
+		(property "Reference" "#FLG06"
 			(at 84.48 19.32 0)
 			(hide yes)
@@
 			(project "AP_RACK16"
 				(path "/8e2a4c6d-0f1b-4d3e-9a5c-7b9d1f3e5a64"
-					(reference "#FLG05")
+					(reference "#FLG06")
 					(unit 1)
 				)
