File: hardware/ap-electric/in16/kicad/AP_IN16.kicad_pcb (KiCad board)
At the start: 2 copper layers, 176 x 100 mm, 208 parts, among them J1 VIN 12-30V, J2 USB-C, J3 KF128-5.08-3P, J4 KF128-5.08-3P, J5 KF128-5.08-3P, J6 KF128-5.08-3P, J7 KF128-5.08-3P, J8 KF128-5.08-3P, SW1 MODO, SW2 RESET, U1 LMR16006XDDC, U2 AP63203WU, U3 ESP32-C3-WROOM-02, U4 USBLC6-2SC6, U5 SP3485EN, U6 TCA9554PWR, U7 TCA9554PWR, U9 TCA9554PWR

Commit message: AP Rack IN16 y AI8: generadores, IN16 cerrada (ERC/DRC 0), AI8 en ruteo
Co-Authored-By: Claude Sonnet 5.5 <noreply@anthropic.com>
Claude-Session: https://claude.ai/code/session_01WVk3oGwfQfGTmAT2PMp8oW
Routing:
- net /GND: track 0.00 -> 748.4 mm, vias 0 -> 420
- net /3V3: track 0.00 -> 434.2 mm, vias 0 -> 11
- net /COMI: track 0.00 -> 350.0 mm, vias 0 -> 1
- net /V24: track 0.00 -> 232.9 mm, vias 0 -> 4
- net /SCL: track 0.00 -> 179.0 mm, vias 0 -> 10
- net /SDA: track 0.00 -> 168.7 mm, vias 0 -> 5
- net /INT: track 0.00 -> 140.9 mm, vias 0 -> 3
- net /RSA: track 0.00 -> 129.1 mm, vias 0 -> 4
- net /RSB: track 0.00 -> 128.6 mm, vias 0 -> 4
- net /SENSE_I: track 0.00 -> 127.4 mm, vias 0 -> 3
- net /SENSE_O: track 0.00 -> 110.1 mm, vias 0 -> 4
- net /V5: track 0.00 -> 107.0 mm, vias 0 -> 2
- net /RS_DE: track 0.00 -> 98.2 mm, vias 0 -> 2
- net /RS_RX: track 0.00 -> 97.2 mm
- net /RS_TX: track 0.00 -> 95.4 mm
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- added copper zone on B.Cu, net /GND
- added copper zone on F.Cu, net /GND
Other:
- board text added: "+V 0V"
- board text added: "AP ELECTRIC AP RACK IN16 rev A - CONCEPTO. 16 entradas 12-30 V. SENSE/A/B: solo AP LINK, no AP BUS."
- board text added: "AP ELECTRIC INDUSTRIAL AP RACK IN16 rev A"
- board text added: "ENTRA"
- board text added: "MODULO 8 4 2 1"
- board text added: "RUN FALLA COM CABEZA"
- board text added: "SIGUE"
