File: hardware/ap-electric/ai8/kicad/AP_AI8.kicad_pcb (KiCad board)
At the start: 2 copper layers, 176 x 100 mm, 146 parts, among them J1 VIN 12-30V, J10 KF128-5.08-3P, J11 KF128-5.08-3P, J12 KF128-5.08-3P, J13 KF128-5.08-3P, J2 USB-C, J6 KF128-5.08-3P, J7 KF128-5.08-3P, J8 KF128-5.08-3P, J9 KF128-5.08-3P, SW1 MODO, SW2 RESET, U1 LMR16006XDDC, U2 AP63203WU, U3 ESP32-C3-WROOM-02, U4 USBLC6-2SC6, U5 SP3485EN, U6 ADS1115IDGSR, U7 ADS1115IDGSR, U9 TCA9554PWR

Commit message: AP Rack IN16: documento, vistas y revisión de direcciones I2C
Co-Authored-By: Claude Sonnet 5.5 <noreply@anthropic.com>
Claude-Session: https://claude.ai/code/session_01WVk3oGwfQfGTmAT2PMp8oW
Parts:
- removed the RB1 at (141.0, 121.0) (x2)
- removed the RB2 at (158.2, 121.0) (x2)
- added RB1: 56k, Resistor_SMD:R_0603_1608Metric, F.Cu at (141.0, 121.0)
- added RB1: 10k, Resistor_SMD:R_0603_1608Metric, F.Cu at (141.0, 121.0)
- added RB2 (x2): 10k, Resistor_SMD:R_0603_1608Metric, F.Cu at (158.2, 121.0)

Commit message: Web nueva (cadena de módulos, panel en vivo, íconos, tema) y placa AP Rack AI8 cerrada por software
- index.html rediseñado: constructor de cadena AP LINK con cables, totales y tabla de direcciones, panel HMI, tema claro/oscuro
- AI8: puentes JP4-JP11, ERC/DRC/paridad 0, pedido sin errores, renders y LEEME
- prueba_sitio.cjs y verificar_todo con IN16/AI8

Co-Authored-By: Claude Sonnet 5.5 <noreply@anthropic.com>
Claude-Session: https://claude.ai/code/session_01WVk3oGwfQfGTmAT2PMp8oW
Parts:
- removed JM1, JM2, JM3, JM4, JM5, JM6, JM7, JM8: 4-20mA, Jumper:SolderJumper-2_P1.3mm_Open_RoundedPad1.0x1.5mm
- removed the RB1 at (141.0, 121.0) (x2)
- removed the RB2 at (158.2, 121.0) (x2)
- removed RB3, RB4, RB5, RB6, RB7, RB8: 10k, Resistor_SMD:R_0603_1608Metric
- added JP10: 4-20mA, Jumper:SolderJumper-2_P1.3mm_Open_RoundedPad1.0x1.5mm, F.Cu at (246.2, 130.0)
- added JP11: 4-20mA, Jumper:SolderJumper-2_P1.3mm_Open_RoundedPad1.0x1.5mm, F.Cu at (263.4, 130.0)
- added JP4: 4-20mA, Jumper:SolderJumper-2_P1.3mm_Open_RoundedPad1.0x1.5mm, F.Cu at (143.0, 130.0)
- added JP5: 4-20mA, Jumper:SolderJumper-2_P1.3mm_Open_RoundedPad1.0x1.5mm, F.Cu at (160.2, 130.0)
- added JP6: 4-20mA, Jumper:SolderJumper-2_P1.3mm_Open_RoundedPad1.0x1.5mm, F.Cu at (177.4, 130.0)
- added JP7: 4-20mA, Jumper:SolderJumper-2_P1.3mm_Open_RoundedPad1.0x1.5mm, F.Cu at (194.6, 130.0)
- added JP8: 4-20mA, Jumper:SolderJumper-2_P1.3mm_Open_RoundedPad1.0x1.5mm, F.Cu at (211.8, 130.0)
- added JP9: 4-20mA, Jumper:SolderJumper-2_P1.3mm_Open_RoundedPad1.0x1.5mm, F.Cu at (229.0, 130.0)
- added RB1: 56k, Resistor_SMD:R_0603_1608Metric, F.Cu at (168.0, 181.5)
- added RB2: 10k, Resistor_SMD:R_0603_1608Metric, F.Cu at (172.5, 181.5)
- added RV1: 10k, Resistor_SMD:R_0603_1608Metric, F.Cu at (141.0, 121.0)
- added RV2: 10k, Resistor_SMD:R_0603_1608Metric, F.Cu at (158.2, 121.0)
- added RV3: 10k, Resistor_SMD:R_0603_1608Metric, F.Cu at (175.4, 121.0)
- added RV4: 10k, Resistor_SMD:R_0603_1608Metric, F.Cu at (192.6, 121.0)
- added RV5: 10k, Resistor_SMD:R_0603_1608Metric, F.Cu at (209.8, 121.0)
- added RV6: 10k, Resistor_SMD:R_0603_1608Metric, F.Cu at (227.0, 121.0)
- added RV7: 10k, Resistor_SMD:R_0603_1608Metric, F.Cu at (244.2, 121.0)
- added RV8: 10k, Resistor_SMD:R_0603_1608Metric, F.Cu at (261.4, 121.0)
Routing:
- net /GND: track 0.00 -> 873.2 mm, vias 0 -> 514
- net /V24: track 0.00 -> 366.9 mm, vias 0 -> 5
- net /3V3: track 0.00 -> 282.4 mm, vias 0 -> 13
- net /SDA: track 0.00 -> 159.2 mm, vias 0 -> 6
- net /SENSE_I: track 0.00 -> 148.8 mm, vias 0 -> 3
- net /SCL: track 0.00 -> 146.9 mm, vias 0 -> 8
- net /RSB: track 0.00 -> 131.2 mm, vias 0 -> 4
- net /SENSE_O: track 0.00 -> 122.4 mm, vias 0 -> 4
- net /RSA: track 0.00 -> 120.0 mm, vias 0 -> 1
- net /VBUS: track 0.00 -> 119.8 mm, vias 0 -> 3
- net /RS_RX: track 0.00 -> 95.5 mm
- net /RS_TX: track 0.00 -> 94.5 mm
- net /RS_DE: track 0.00 -> 94.5 mm, vias 0 -> 2
- net /AN8: track 0.00 -> 89.3 mm
- net /V5: track 0.00 -> 84.6 mm, vias 0 -> 3
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- added copper zone on B.Cu, net /GND
- added copper zone on F.Cu, net /GND
Other:
- board text added: "+V 0V"
- board text added: "AI1"
- board text added: "AI2"
- board text added: "AI3"
- board text added: "AI4"
- board text added: "AI5"
- board text added: "AI6"
- board text added: "AI7"
- board text added: "AI8"
- board text added: "AP ELECTRIC AP RACK AI8 rev A - CONCEPTO. 0-10 V / 4-20 mA. Puente cerrado: NO conectar voltaje. SENSE/A/B: solo AP LINK."
- board text added: "AP ELECTRIC INDUSTRIAL AP RACK AI8 rev A"
- board text added: "ENTRA"
- board text added: "MODULO 8 4 2 1"
- board text added: "RUN FALLA COM CABEZA"
- board text added: "SIGUE"
- board text added: "mA: cerrar JP4-JP11"
