File: hardware/ap-electric/ai8/kicad/AP_AI8.kicad_sch (KiCad schematic)
At the start: 140 parts, among them J1 VIN 12-30V, J10 KF128-5.08-3P, J11 KF128-5.08-3P, J12 KF128-5.08-3P, J13 KF128-5.08-3P, J2 USB-C, J6 KF128-5.08-3P, J7 KF128-5.08-3P, J8 KF128-5.08-3P, J9 KF128-5.08-3P, SW1 MODO, SW2 RESET, U1 LMR16006XDDC, U2 AP63203WU, U3 ESP32-C3-WROOM-02, U4 USBLC6-2SC6, U5 SP3485EN, U6 ADS1115IDGSR, U7 ADS1115IDGSR, U9 TCA9554PWR

Commit message: Web nueva (cadena de módulos, panel en vivo, íconos, tema) y placa AP Rack AI8 cerrada por software
- index.html rediseñado: constructor de cadena AP LINK con cables, totales y tabla de direcciones, panel HMI, tema claro/oscuro
- AI8: puentes JP4-JP11, ERC/DRC/paridad 0, pedido sin errores, renders y LEEME
- prueba_sitio.cjs y verificar_todo con IN16/AI8

Co-Authored-By: Claude Sonnet 5.5 <noreply@anthropic.com>
Claude-Session: https://claude.ai/code/session_01WVk3oGwfQfGTmAT2PMp8oW
Parts:
- removed JM1, JM2, JM3, JM4, JM5, JM6, JM7, JM8: 4-20mA, Jumper:SolderJumper-2_P1.3mm_Open_RoundedPad1.0x1.5mm, symbol Jumper:SolderJumper_2_Open
- removed RB3, RB4, RB5, RB6, RB7, RB8: 10k, Resistor_SMD:R_0603_1608Metric, symbol Device:R
- added JP10, JP11, JP4, JP5, JP6, JP7, JP8, JP9: 4-20mA, Jumper:SolderJumper-2_P1.3mm_Open_RoundedPad1.0x1.5mm, symbol Jumper:SolderJumper_2_Open
- added RV1, RV2, RV3, RV4, RV5, RV6, RV7, RV8: 10k, Resistor_SMD:R_0603_1608Metric, symbol Device:R
- RB1: value 10k -> 56k; Funcion Divisor canal 1 -> Divisor: 0.765 V x 6.6 = 5.05 V
- RB2: Funcion Divisor canal 2 -> Divisor
Connections:
- net GND: now also JP10.2 (B), JP11.2 (B), JP4.2 (B), JP5.2 (B), JP6.2 (B), JP7.2 (B), JP8.2 (B), JP9.2 (B), RV1.2, RV2.2, RV3.2, RV4.2, RV5.2, RV6.2, RV7.2, RV8.2; no longer RB1.2
- net MA1: now also JP4.1 (A)
- net MA2: now also JP5.1 (A)
- net MA3: now also JP6.1 (A)
- net MA4: now also JP7.1 (A)
- net MA5: now also JP8.1 (A)
- net MA6: now also JP9.1 (A)
- net MA7: now also JP10.1 (A)
- net MA8: now also JP11.1 (A)
- net ND1: now also RV1.1; no longer RB1.1
- net ND2: now also RV2.1; no longer RB2.1
- net ND3: now also RV3.1
- net ND4: now also RV4.1
- net ND5: now also RV5.1
- net ND6: now also RV6.1
- net ND7: now also RV7.1
- net ND8: now also RV8.1
Other:
- note added: "AP Electric Industrial · AP Rack AI8 rev A (CONCEPTO): 2 x ADS1115 (I2C 0x48, 0x49), 8 entradas 0-10 V (22k/10k) o 4-20 mA (150 ohm con JP4-JP11), SP3485 + 2 x JST XH4 (AP LINK), ESP32-C3. No aislado."
- note removed: "AP Electric Industrial · AP Rack AI8 rev A (CONCEPTO): 2 x ADS1115 (I2C 0x48, 0x49), 8 entradas 0-10 V (22k/10k) o 4-20 mA (150 ohm con JMn), SP3485 + 2 x JST XH4 (AP LINK), ESP32-C3. No aislado."
Changed lines of the file:
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@@
 		(on_board yes)
 		(dnp no)
-		(property "Reference" "RB1"
+		(property "Reference" "RV1"
 			(at 163.22 496.84 0)
 			(effects
@@
 			(project "AP_AI8"
 				(path "/9b1d3f5a-7c2e-4b4d-8a6f-0e2c4a6b8d10"
-					(reference "RB1")
+					(reference "RV1")
 					(unit 1)
 				)
@@
 		(on_board yes)
 		(dnp no)
-		(property "Reference" "JM1"
+		(property "Reference" "JP4"
 			(at 28.67 532.74 0)
 			(effects
@@
 			(project "AP_AI8"
 				(path "/9b1d3f5a-7c2e-4b4d-8a6f-0e2c4a6b8d10"
-					(reference "JM1")
+					(reference "JP4")
 					(unit 1)
 				)
@@
 		(on_board yes)
 		(dnp no)
-		(property "Reference" "RB2"
+		(property "Reference" "RV2"
 			(at 163.22 534.94 0)
 			(effects
@@
 			(project "AP_AI8"
 				(path "/9b1d3f5a-7c2e-4b4d-8a6f-0e2c4a6b8d10"
-					(reference "RB2")
+					(reference "RV2")
 					(unit 1)
 				)
@@
 		(on_board yes)
 		(dnp no)
-		(property "Reference" "JM2"
+		(property "Reference" "JP5"
 			(at 28.67 570.84 0)
 			(effects
@@
 			(project "AP_AI8"
 				(path "/9b1d3f5a-7c2e-4b4d-8a6f-0e2c4a6b8d10"
-					(reference "JM2")
+					(reference "JP5")
 					(unit 1)
 				)
@@
 		(on_board yes)
 		(dnp no)
-		(property "Reference" "RB3"
+		(property "Reference" "RV3"
 			(at 163.22 573.04 0)
 			(effects
@@
 			(project "AP_AI8"
 				(path "/9b1d3f5a-7c2e-4b4d-8a6f-0e2c4a6b8d10"
-					(reference "RB3")
+					(reference "RV3")
 					(unit 1)
 				)
@@
 		(on_board yes)
 		(dnp no)
-		(property "Reference" "JM3"
+		(property "Reference" "JP6"
 			(at 28.67 608.94 0)
 			(effects
@@
 			(project "AP_AI8"
 				(path "/9b1d3f5a-7c2e-4b4d-8a6f-0e2c4a6b8d10"
-					(reference "JM3")
+					(reference "JP6")
 					(unit 1)
 				)
@@
 		(on_board yes)
 		(dnp no)
-		(property "Reference" "RB4"
+		(property "Reference" "RV4"
 			(at 163.22 611.14 0)
 			(effects
@@
 			(project "AP_AI8"
 				(path "/9b1d3f5a-7c2e-4b4d-8a6f-0e2c4a6b8d10"
-					(reference "RB4")
+					(reference "RV4")
 					(unit 1)
 				)
@@
 		(on_board yes)
 		(dnp no)
-		(property "Reference" "JM4"
+		(property "Reference" "JP7"
 			(at 28.67 647.04 0)
 			(effects
@@
 			(project "AP_AI8"
 				(path "/9b1d3f5a-7c2e-4b4d-8a6f-0e2c4a6b8d10"
-					(reference "JM4")
+					(reference "JP7")
 					(unit 1)
 				)
@@
 		(on_board yes)
 		(dnp no)
-		(property "Reference" "RB5"
+		(property "Reference" "RV5"
 			(at 163.22 649.24 0)
 			(effects
@@
 			(project "AP_AI8"
 				(path "/9b1d3f5a-7c2e-4b4d-8a6f-0e2c4a6b8d10"
-					(reference "RB5")
+					(reference "RV5")
 					(unit 1)
 				)
@@
 		(on_board yes)
 		(dnp no)
-		(property "Reference" "JM5"
+		(property "Reference" "JP8"
 			(at 28.67 685.14 0)
 			(effects
@@
 			(project "AP_AI8"
 				(path "/9b1d3f5a-7c2e-4b4d-8a6f-0e2c4a6b8d10"
-					(reference "JM5")
+					(reference "JP8")
 					(unit 1)
 				)
@@
 		(on_board yes)
 		(dnp no)
-		(property "Reference" "RB6"
+		(property "Reference" "RV6"
 			(at 163.22 687.34 0)
 			(effects
@@
 			(project "AP_AI8"
 				(path "/9b1d3f5a-7c2e-4b4d-8a6f-0e2c4a6b8d10"
-					(reference "RB6")
+					(reference "RV6")
 					(unit 1)
 				)
@@
 		(on_board yes)
 		(dnp no)
-		(property "Reference" "JM6"
+		(property "Reference" "JP9"
 			(at 28.67 723.24 0)
 			(effects
@@
 			(project "AP_AI8"
 				(path "/9b1d3f5a-7c2e-4b4d-8a6f-0e2c4a6b8d10"
-					(reference "JM6")
+					(reference "JP9")
 					(unit 1)
 				)
@@
 		(on_board yes)
 		(dnp no)
-		(property "Reference" "RB7"
+		(property "Reference" "RV7"
 			(at 163.22 725.44 0)
 			(effects
@@
 			(project "AP_AI8"
 				(path "/9b1d3f5a-7c2e-4b4d-8a6f-0e2c4a6b8d10"
-					(reference "RB7")
+					(reference "RV7")
 					(unit 1)
 				)
@@
 		(on_board yes)
 		(dnp no)
-		(property "Reference" "JM7"
+		(property "Reference" "JP10"
 			(at 28.67 761.34 0)
 			(effects
@@
 			(project "AP_AI8"
 				(path "/9b1d3f5a-7c2e-4b4d-8a6f-0e2c4a6b8d10"
-					(reference "JM7")
+					(reference "JP10")
 					(unit 1)
 				)
@@
 		(on_board yes)
 		(dnp no)
-		(property "Reference" "RB8"
+		(property "Reference" "RV8"
 			(at 163.22 763.54 0)
 			(effects
@@
 			(project "AP_AI8"
 				(path "/9b1d3f5a-7c2e-4b4d-8a6f-0e2c4a6b8d10"
-					(reference "RB8")
+					(reference "RV8")
 					(unit 1)
 				)
@@
 		(on_board yes)
 		(dnp no)
-		(property "Reference" "JM8"
+		(property "Reference" "JP11"
 			(at 28.67 799.44 0)
 			(effects
@@
 			(project "AP_AI8"
 				(path "/9b1d3f5a-7c2e-4b4d-8a6f-0e2c4a6b8d10"
-					(reference "JM8")
+					(reference "JP11")
 					(unit 1)
 				)
@@
 		)
 	)
-	(symbol
-		(lib_id "power:PWR_FLAG")
-		(at 81.28 20.32 0)
-		(unit 1)
-		(exclude_from_sim no)
-		(in_bom no)
-		(on_board no)
-		(dnp no)
-		(property "Reference" "#FLG06"
-			(at 84.48 19.32 0)
-			(hide yes)
-			(effects
-				(font
-					(size 1.27 1.27)
-				)
-				(justify left)
-			)
-		)
-		(property "Value" "PWR_FLAG"
-			(at 84.48 21.92 0)
-			(effects
-				(font
-					(size 1.27 1.27)
-				)
-				(justify left)
-			)
-		)
-		(property "Footprint" ""
-			(at 81.28 20.32 0)
-			(hide yes)
-			(effects
-				(font
-					(size 1.27 1.27)
-				)
-				(justify left)
-			)
-		)
-		(property "Datasheet" "~"
-			(at 81.28 20.32 0)
-			(hide yes)
-			(effects
-				(font
-					(size 1.27 1.27)
-				)
-				(justify left)
-			)
-		)
-		(property "Description" "Bandera de alimentación para ERC"
-			(at 81.28 20.32 0)
-			(hide yes)
-			(effects
-				(font
-					(size 1.27 1.27)
-				)
-				(justify left)
-			)
-		)
-		(pin "1"
-		)
-		(instances
-			(project "AP_AI8"
-				(path "/9b1d3f5a-7c2e-4b4d-8a6f-0e2c4a6b8d10"
-					(reference "#FLG06")
-					(unit 1)
-				)
-			)
-		)
-	)
-	(wire
-		(pts
-			(xy 81.28 20.32)
-			(xy 81.28 22.86)
-		)
-		(stroke
-			(width 0)
-			(type default)
-		)
-	)
-	(label "COMI"
-		(at 81.28 22.86 0)
-		(fields_autoplaced yes)
-		(effects
-			(font
-				(size 1.27 1.27)
-			)
-			(justify left bottom)
-		)
-	)
-	(text "AP Electric Industrial · AP Rack AI8 rev A (CONCEPTO): 2 x ADS1115 (I2C 0x48, 0x49), 8 entradas 0-10 V (22k/10k) o 4-20 mA (150 ohm con JMn),\nSP3485 + 2 x JST XH4 (AP LINK), ESP32-C3. No aislado."
+	(text "AP Electric Industrial · AP Rack AI8 rev A (CONCEPTO): 2 x ADS1115 (I2C 0x48, 0x49), 8 entradas 0-10 V (22k/10k) o 4-20 mA (150 ohm con JP4-JP11),\nSP3485 + 2 x JST XH4 (AP LINK), ESP32-C3. No aislado."
 		(exclude_from_sim no)
 		(at 150 15 0)
