File: hardware/ap-electric/plcb/kicad/AP_PLC_C24B.kicad_pcb (KiCad board)
At the start: 2 copper layers, 200 x 100 mm, 299 parts, among them J1 VIN 12-30V, J10 KF128-5.08-3P, J11 KF128-5.08-3P, J12 KF128-5.08-3P, J13 KF128-5.08-3P, J14 HR911105A, J15 BAT, J16 KF128-5.08-3P, J2 USB-C, J3 KF128-5.08-3P, J4 KF128-5.08-3P, J5 KF128-5.08-3P, J6 KF128-5.08-3P, J7 KF128-5.08-3P, J8 KF128-5.08-3P, J9 KF128-5.08-3P, Q1 NCV8406ASTT3G, Q10 NCV8406ASTT3G, Q11 NCV8406ASTT3G, Q12 NCV8406ASTT3G, Q2 NCV8406ASTT3G, Q3 NCV8406ASTT3G, Q4 NCV8406ASTT3G, Q5 NCV8406ASTT3G, Q6 NCV8406ASTT3G, Q7 NCV8406ASTT3G, Q8 NCV8406ASTT3G, Q9 NCV8406ASTT3G, SW1 MODO, SW2 RESET, SW3 RUN/STOP, U1 LMR16006XDDC, U10 74HCT125D, U11 74HCT125D, U12 74HCT125D, U15 TCA9554PWR, U16 W5500, U17 PCF8563T/5,518, U18 SP3485EN, U2 AP63203WU, U3 ESP32-S3-WROOM-1, U4 USBLC6-2SC6, U5 SP3485EN, U6 TCA9554PWR, U7 TCA9554PWR, U8 TCA9554PWR, U9 TCA9554PWR, Y1 25MHz, Y2 32.768kHz 12.5pF

Commit message: AP PLC C24 rev B: sin interrupción de expansores, expansor de LED junto a su fila; ruteo sigue sin cerrar (6 pendientes)
Co-Authored-By: Claude Sonnet 5.5 <noreply@anthropic.com>
Claude-Session: https://claude.ai/code/session_01WVk3oGwfQfGTmAT2PMp8oW
Parts:
- removed R5: 10k, Resistor_SMD:R_0603_1608Metric
- moved TP10 77.8 mm to (287.0, 198.0)
- moved TP9 77.1 mm to (282.0, 198.0)
- moved TP8 68.3 mm to (277.0, 198.0)
- moved TP7 67.6 mm to (272.0, 198.0)
- moved U9 20.1 mm to (228.0, 152.0)
- moved C18 8.73 mm to (221.5, 152.0)
Connections:
- U15 pad 13: /INT -> unconnected-(U15-~{INT}-Pad13)
- U3 pad 18: /INT -> unconnected-(U3-IO10-Pad18)
- U8 pad 13: /INT -> unconnected-(U8-~{INT}-Pad13)
