File: hardware/ap-electric/plcb/kicad/AP_PLC_C24B.kicad_sch (KiCad schematic)
At the start: 295 parts, among them J1 VIN 12-30V, J10 KF128-5.08-3P, J11 KF128-5.08-3P, J12 KF128-5.08-3P, J13 KF128-5.08-3P, J14 HR911105A, J15 BAT, J16 KF128-5.08-3P, J2 USB-C, J3 KF128-5.08-3P, J4 KF128-5.08-3P, J5 KF128-5.08-3P, J6 KF128-5.08-3P, J7 KF128-5.08-3P, J8 KF128-5.08-3P, J9 KF128-5.08-3P, Q1 NCV8406ASTT3G, Q10 NCV8406ASTT3G, Q11 NCV8406ASTT3G, Q12 NCV8406ASTT3G, Q2 NCV8406ASTT3G, Q3 NCV8406ASTT3G, Q4 NCV8406ASTT3G, Q5 NCV8406ASTT3G, Q6 NCV8406ASTT3G, Q7 NCV8406ASTT3G, Q8 NCV8406ASTT3G, Q9 NCV8406ASTT3G, SW1 MODO, SW2 RESET, SW3 RUN/STOP, U1 LMR16006XDDC, U10 74HCT125D, U11 74HCT125D, U12 74HCT125D, U15 TCA9554PWR, U16 W5500, U17 PCF8563T/5,518, U18 SP3485EN, U2 AP63203WU, U3 ESP32-S3-WROOM-1, U4 USBLC6-2SC6, U5 SP3485EN, U6 TCA9554PWR, U7 TCA9554PWR, U8 TCA9554PWR, U9 TCA9554PWR, Y1 25MHz, Y2 32.768kHz 12.5pF

Commit message: AP PLC C24 rev B: sin interrupción de expansores, expansor de LED junto a su fila; ruteo sigue sin cerrar (6 pendientes)
Co-Authored-By: Claude Sonnet 5.5 <noreply@anthropic.com>
Claude-Session: https://claude.ai/code/session_01WVk3oGwfQfGTmAT2PMp8oW
Parts:
- removed R5: 10k, Resistor_SMD:R_0603_1608Metric, symbol Device:R
- U3: Funcion IO4/IO5/IO6 = RS-485 de Modbus, IO7 = tensión de entrada, IO8/IO9 = I2C, IO10 = interrupción de entradas, IO11/IO12 = SENSE, IO16/IO17/IO18 = AP LINK, IO38-IO42 = W5500, IO2 = reset del W5500, IO0 = MODO -> IO4/IO5/IO6 = RS-485 de Modbus, IO7 = tensión de entrada, IO8/IO9 = I2C, IO10 sin uso (la interrupción de los expansores no se cablea: el programa consulta cada 5 ms), IO11/IO12 = SENSE, IO16/IO17/IO18 = AP LINK, IO38-IO42 = W5500, IO2 = reset del W5500, IO0 = MODO
Connections:
- removed net INT: U15.13 (~{INT}), U3.18 (IO10), U8.13 (~{INT})
- no-connect marks 37 -> 40
Other:
- moved on the sheet: C13, C14, C15, C16, C17, C18, C19, C22, C23, C24, C25, C26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
